File: adc board/haasoscope_pro_adc_board - no blind.sch (EAGLE design)
At the start: 164 parts, among them IC1 ADC12DL2500ACF, IC2 SN74AVC4T774PWR, J1 8pin, J10 8pin, J11 8pin, J12 8pin, J13 8pin, J16 8pin, J17 8pin, J2 8pin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

Commit message: fix pins for bottom rows of fpga
Parts:
- renumbered A14_CLKOUT2- to B13_CLKOUT2-, B14_CLKOUT2+ to D11_CLKOUT2+
Connections:
- net A10 renamed B11
- net A14_CLKOUT2N renamed B13_CLKOUT2N
- net B14_CLKOUT2P renamed D11_CLKOUT2P
- net C6 renamed D5
- net D11 renamed B14
- net E11_SYNCSE renamed F10_SYNCSE
- net E7 renamed D6
- net G11 renamed F9
- net A7: now also PINOUT2.5, X2-15.S; no longer PINOUT1.8, X2-16.S
- net C8: now also PINOUT2.8, X1-16.S; no longer PINOUT1.4, X1-15.S
- net D8: now also PINOUT1.4, X1-15.S; no longer PINOUT2.8, X1-16.S
- net E10: now also PINOUT2.3, X2-2.S; no longer PINOUT2.7, X2-1.S
- net E6: now also PINOUT1.8, X2-16.S; no longer PINOUT2.5, X2-15.S
- net E9: now also PINOUT2.7, X2-1.S; no longer PINOUT2.3, X2-2.S
Other:
- note added: "A10"
- note added: "A14"
- note added: "C6"
- note added: "DIFF44!"
- note added: "E11"
- note added: "E7"
- note added: "G11"
- note removed: "B11"
- note removed: "B13"
- note removed: "D5"
- note removed: "D6"
- note removed: "F10"
- note removed: "F9"
