File: fpga board/haasoscope_pro_fpga_board.brd (EAGLE design)
At the start: 155.5 x 111.5 mm, 406 parts, among them IC1 EP4CE30F23C6N, IC2 EPCQ16ASI8N, J1 2x5, SW1 SKQGADE010, SW2 SKQGADE010, U1 AMS1117-3.3, U2 AMS1117-2.5, U3 AMS1117-1.2, Y1 OSCILLATORSMD-5X3

Commit message: pull tms and tdi up to 3v3
Parts:
- added R10, R11: 10k, FlashPCB_Resistors:RES-0402
Connections:
- net 3V3: now also R10.P$2, R11.P$2
- net TDI: now also R11.P$1
- net TMS: now also R10.P$1
Routing:
- net 3V3: track 337.8 -> 349.2 mm
- net TMS: track 72.9 -> 83.2 mm
- net TDI: track 101.3 -> 111.4 mm
Changed lines of the file:
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@@
 <drawing>
 <settings>
-<setting alwaysvectorfont="yes"/>
+<setting alwaysvectorfont="no"/>
 <setting verticaltext="up"/>
 </settings>
@@
 <layers>
 <layer number="1" name="top" color="12" fill="1" visible="yes" active="yes"/>
-<layer number="2" name="topgnd" color="12" fill="5" visible="no" active="yes"/>
+<layer number="2" name="topgnd" color="12" fill="5" visible="yes" active="yes"/>
 <layer number="3" name="sig2" color="4" fill="1" visible="yes" active="yes"/>
-<layer number="4" name="sig2gnd" color="4" fill="5" visible="no" active="yes"/>
-<layer number="5" name="pow1" color="7" fill="8" visible="no" active="yes"/>
+<layer number="4" name="sig2gnd" color="4" fill="5" visible="yes" active="yes"/>
+<layer number="5" name="pow1" color="7" fill="8" visible="yes" active="yes"/>
 <layer number="6" name="pwr2" color="16" fill="8" visible="no" active="no"/>
 <layer number="7" name="sig7gnd" color="15" fill="5" visible="no" active="no"/>
@@
 <layer number="10" name="sig7" color="31" fill="1" visible="no" active="no"/>
 <layer number="11" name="sig6gnd" color="11" fill="5" visible="no" active="no"/>
-<layer number="12" name="pow2" color="30" fill="8" visible="no" active="yes"/>
-<layer number="13" name="sig4gnd" color="1" fill="5" visible="no" active="yes"/>
+<layer number="12" name="pow2" color="30" fill="8" visible="yes" active="yes"/>
+<layer number="13" name="sig4gnd" color="1" fill="5" visible="yes" active="yes"/>
 <layer number="14" name="sig4" color="1" fill="1" visible="yes" active="yes"/>
-<layer number="15" name="sig5gnd" color="5" fill="5" visible="no" active="yes"/>
+<layer number="15" name="sig5gnd" color="5" fill="5" visible="yes" active="yes"/>
 <layer number="16" name="sig5" color="5" fill="1" visible="yes" active="yes"/>
 <layer number="17" name="Pads" color="2" fill="1" visible="yes" active="yes"/>
@@
 <layer number="49" name="Reference" color="7" fill="1" visible="no" active="yes"/>
 <layer number="50" name="dxf" color="7" fill="1" visible="no" active="no"/>
-<layer number="51" name="tDocu" color="7" fill="1" visible="no" active="yes"/>
-<layer number="52" name="bDocu" color="7" fill="1" visible="no" active="yes"/>
+<layer number="51" name="tDocu" color="7" fill="1" visible="yes" active="yes"/>
+<layer number="52" name="bDocu" color="7" fill="1" visible="yes" active="yes"/>
 <layer number="53" name="tGND_GNDA" color="7" fill="9" visible="no" active="no"/>
 <layer number="54" name="bGND_GNDA" color="1" fill="9" visible="no" active="no"/>
@@
 <attribute name="POPULARITY" value="64" x="38.5" y="-80.5" size="1.778" layer="27" display="off"/>
 </element>
+<element name="R10" library="FlashPCB_Resistors" package="RES-0402" value="10k" x="-28" y="-11.5" smashed="yes">
+<attribute name="NAME" x="-29.27" y="-10" size="0.8128" layer="25" font="vector"/>
+<attribute name="VALUE" x="-29.27" y="-11" size="0.8128" layer="27" font="vector"/>
+</element>
+<element name="R11" library="FlashPCB_Resistors" package="RES-0402" value="10k" x="-28" y="-14.5" smashed="yes">
+<attribute name="NAME" x="-29.27" y="-13" size="0.8128" layer="25" font="vector"/>
+<attribute name="VALUE" x="-29.27" y="-14" size="0.8128" layer="27" font="vector"/>
+</element>
 </elements>
 <signals>
@@
 <wire x1="-34.5" y1="14.5" x2="-38.5" y2="10.5" width="0.1524" layer="1"/>
 <wire x1="-33" y1="14.5" x2="-34.5" y2="14.5" width="0.1524" layer="1"/>
-<wire x1="-35.25" y1="-10.75" x2="-35.25" y2="-11.25" width="0.1524" layer="1"/>
-<wire x1="-36.5" y1="-9.5" x2="-35.25" y2="-10.75" width="0.1524" layer="1"/>
-<wire x1="-36.5" y1="0.5" x2="-36.5" y2="-9.5" width="0.1524" layer="1"/>
+<wire x1="-35.25" y1="-10.88" x2="-35.25" y2="-11.25" width="0.1524" layer="1"/>
+<wire x1="-36.5" y1="-9.63" x2="-35.5" y2="-10.63" width="0.1524" layer="1"/>
+<wire x1="-35.5" y1="-10.63" x2="-35.25" y2="-10.88" width="0.1524" layer="1"/>
+<wire x1="-36.5" y1="0.5" x2="-36.5" y2="-9.63" width="0.1524" layer="1"/>
 <wire x1="-38" y1="2" x2="-36.5" y2="0.5" width="0.1524" layer="1"/>
 <wire x1="-38" y1="5.5" x2="-38" y2="2" width="0.1524" layer="1"/>
@@
 <via x="14" y="18.5" extent="1-16" drill="0.2"/>
 <via x="22" y="54.5" extent="1-16" drill="0.2"/>
+<contactref element="R10" pad="P$2"/>
+<contactref element="R11" pad="P$2"/>
+<wire x1="-27.5" y1="-14.5" x2="-27.5" y2="-11.5" width="0.1524" layer="1"/>
+<wire x1="-27.5" y1="-11.5" x2="-28.37" y2="-10.63" width="0.1524" layer="1"/>
+<wire x1="-28.37" y1="-10.63" x2="-35.5" y2="-10.63" width="0.1524" layer="1"/>
 </signal>
 <signal name="IO153">
@@
 <wire x1="-37.75" y1="-14" x2="-37.77" y2="-14" width="0.0889" layer="5"/>
 <via x="2.75" y="11.25" extent="1-16" drill="0.2"/>
+<contactref element="R10" pad="P$1"/>
+<wire x1="-28.5" y1="-11.5" x2="-29.733" y2="-12.733" width="0.1524" layer="1"/>
+<wire x1="-36.503" y1="-12.733" x2="-37.77" y2="-14" width="0.1524" layer="1"/>
+<wire x1="-29.733" y1="-12.733" x2="-36.503" y2="-12.733" width="0.1524" layer="1"/>
 </signal>
 <signal name="TCK">
@@
 <wire x1="18.57365" y1="12.1778" x2="17.8222" y2="12.1778" width="0.0889" layer="3"/>
 <wire x1="24.5745625" y1="12.04925" x2="18.7022" y2="12.04925" width="0.0889" layer="3"/>
-<wire x1="-37.77" y1="-17.8601" x2="-37.77" y2="-19.08" width="0.0889" layer="3"/>
-<wire x1="-36.83655" y1="-16.92665" x2="-37.77" y2="-17.8601" width="0.0889" layer="3"/>
 <wire x1="25" y1="12" x2="25.5" y2="12.5" width="0.0889" layer="5"/>
 <wire x1="14.5" y1="12" x2="25" y2="12" width="0.0889" layer="5"/>
@@
 <wire x1="-37.75" y1="-19" x2="-37.77" y2="-19.08" width="0.0889" layer="14"/>
 <via x="12" y="14.5" extent="1-16" drill="0.2"/>
+<contactref element="R11" pad="P$1"/>
+<wire x1="-33.19" y1="-14.5" x2="-28.5" y2="-14.5" width="0.1524" layer="1"/>
+<wire x1="-37.77" y1="-19.08" x2="-36.503" y2="-17.813" width="0.1524" layer="1"/>
+<wire x1="-33.977" y1="-15.287" x2="-33.19" y2="-14.5" width="0.1524" layer="1"/>
+<wire x1="-36.503" y1="-17.813" x2="-36.503" y2="-15.287" width="0.1524" layer="1"/>
+<wire x1="-36.503" y1="-15.287" x2="-33.977" y2="-15.287" width="0.1524" layer="1"/>
 </signal>
 <signal name="IO148">

Commit message: pull down tck to gnd with 1k
Parts:
- added R12: 1k, FlashPCB_Resistors:RES-0402
Connections:
- net GND: now also R12.P$1
- net TCK: now also R12.P$2
Routing:
- net TCK: track 73.3 -> 82.0 mm
- net GND: track 119.5 -> 128.2 mm
Changed lines of the file:
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@@
 <drawing>
 <settings>
-<setting alwaysvectorfont="no"/>
+<setting alwaysvectorfont="yes"/>
 <setting verticaltext="up"/>
 </settings>
@@
 <layers>
 <layer number="1" name="top" color="12" fill="1" visible="yes" active="yes"/>
-<layer number="2" name="topgnd" color="12" fill="5" visible="yes" active="yes"/>
+<layer number="2" name="topgnd" color="12" fill="5" visible="no" active="yes"/>
 <layer number="3" name="sig2" color="4" fill="1" visible="yes" active="yes"/>
-<layer number="4" name="sig2gnd" color="4" fill="5" visible="yes" active="yes"/>
-<layer number="5" name="pow1" color="7" fill="8" visible="yes" active="yes"/>
+<layer number="4" name="sig2gnd" color="4" fill="5" visible="no" active="yes"/>
+<layer number="5" name="pow1" color="7" fill="8" visible="no" active="yes"/>
 <layer number="6" name="pwr2" color="16" fill="8" visible="no" active="no"/>
 <layer number="7" name="sig7gnd" color="15" fill="5" visible="no" active="no"/>
@@
 <layer number="10" name="sig7" color="31" fill="1" visible="no" active="no"/>
 <layer number="11" name="sig6gnd" color="11" fill="5" visible="no" active="no"/>
-<layer number="12" name="pow2" color="30" fill="8" visible="yes" active="yes"/>
-<layer number="13" name="sig4gnd" color="1" fill="5" visible="yes" active="yes"/>
+<layer number="12" name="pow2" color="30" fill="8" visible="no" active="yes"/>
+<layer number="13" name="sig4gnd" color="1" fill="5" visible="no" active="yes"/>
 <layer number="14" name="sig4" color="1" fill="1" visible="yes" active="yes"/>
-<layer number="15" name="sig5gnd" color="5" fill="5" visible="yes" active="yes"/>
+<layer number="15" name="sig5gnd" color="5" fill="5" visible="no" active="yes"/>
 <layer number="16" name="sig5" color="5" fill="1" visible="yes" active="yes"/>
 <layer number="17" name="Pads" color="2" fill="1" visible="yes" active="yes"/>
@@
 <attribute name="VALUE" x="-29.27" y="-14" size="0.8128" layer="27" font="vector"/>
 </element>
+<element name="R12" library="FlashPCB_Resistors" package="RES-0402" value="1k" x="-36.5" y="-0.5" smashed="yes" rot="R180">
+<attribute name="NAME" x="-35.23" y="-2" size="0.8128" layer="25" font="vector" rot="R180"/>
+<attribute name="VALUE" x="-35.23" y="-1" size="0.8128" layer="27" font="vector" rot="R180"/>
+</element>
 </elements>
 <signals>
@@
 <via x="12" y="20.5" extent="1-16" drill="0.2"/>
 <via x="-34.5" y="8.5" extent="1-16" drill="0.2"/>
+<contactref element="R12" pad="P$1"/>
+<wire x1="-36" y1="-0.5" x2="-35.23" y2="-1.27" width="0.1524" layer="1"/>
+<wire x1="-35.23" y1="-1.27" x2="-35.23" y2="-8.92" width="0.1524" layer="1"/>
 </signal>
 <signal name="5V" class="1">
@@
 <wire x1="-2.91415" y1="12.878525" x2="-2.91415" y2="13.449775" width="0.0889" layer="16"/>
 <wire x1="-6.949775" y1="14.08585" x2="-7.91415" y2="13.121475" width="0.0889" layer="16"/>
+<contactref element="R12" pad="P$2"/>
+<wire x1="-37.77" y1="-1.27" x2="-37.77" y2="-8.92" width="0.1524" layer="1"/>
+<wire x1="-37" y1="-0.5" x2="-37.77" y2="-1.27" width="0.1524" layer="1"/>
 </signal>
 <signal name="NCE">
