File: data board/data board.brd (EAGLE design)
At the start: 47.6 x 32 mm, 41 parts, among them IC1 93LC56B, IC2 FT232HQ, U1 CJT1117-5.0-SOT223, U9 MOSFET-PCHANNEL-SOIC8SOIC8, X3 HUSB238, X6 USBC, Y1 12MHz

Commit message: Revert "v1.1"
This reverts commit 9c2a8abd0e838ea48c804dee952ae91d8fcae4a4.
Parts:
- renumbered U9 to U$9
Changed lines of the file:
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@@
 </element>
 <element name="U1" library="Seeed-IC" library_urn="urn:adsk.eagle:library:470" package="SOT-223" package3d_urn="urn:adsk.eagle:package:32638/1" value="CJT1117-5.0-SOT223" x="-6" y="-1" smashed="yes" rot="R180">
-<attribute name="LCSC" value="C89273" x="-6" y="-1" size="1.778" layer="27" rot="R180" display="off"/>
 <attribute name="MPN" value="CJT1117-5.0" x="7" y="30" size="1.778" layer="27" rot="R180" display="off"/>
 <attribute name="VALUE" x="-12.71" y="-6.645" size="0.8128" layer="21"/>
 </element>
-<element name="U9" library="SparkFun-DiscreteSemi" package="SO08" value="MOSFET-PCHANNEL-SOIC8SOIC8" x="-5" y="17" smashed="yes">
+<element name="U$9" library="SparkFun-DiscreteSemi" package="SO08" value="MOSFET-PCHANNEL-SOIC8SOIC8" x="-5" y="17" smashed="yes">
 <attribute name="LCSC" value="C143671" x="-25" y="-5" size="1.778" layer="27" display="off"/>
 <attribute name="VALUE" x="-13.87" y="21.765" size="0.8128" layer="21"/>
@@
 </signal>
 <signal name="VBUS" class="1">
-<contactref element="U9" pad="1"/>
-<contactref element="U9" pad="2"/>
-<contactref element="U9" pad="3"/>
+<contactref element="U$9" pad="1"/>
+<contactref element="U$9" pad="2"/>
+<contactref element="U$9" pad="3"/>
 <contactref element="R7" pad="P$2"/>
 <contactref element="R9" pad="P$2"/>
@@
 <signal name="VOUT">
 <contactref element="U1" pad="3"/>
-<contactref element="U9" pad="8"/>
-<contactref element="U9" pad="7"/>
-<contactref element="U9" pad="6"/>
-<contactref element="U9" pad="5"/>
+<contactref element="U$9" pad="8"/>
+<contactref element="U$9" pad="7"/>
+<contactref element="U$9" pad="6"/>
+<contactref element="U$9" pad="5"/>
 <contactref element="C17" pad="2"/>
 <contactref element="C18" pad="2"/>
@@
 </signal>
 <signal name="GATE">
-<contactref element="U9" pad="4"/>
+<contactref element="U$9" pad="4"/>
 <contactref element="R9" pad="P$1"/>
 <contactref element="R8" pad="P$2"/>

Commit message: v1.1
Parts:
- renumbered U$9 to U9
Changed lines of the file:
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@@
 </element>
 <element name="U1" library="Seeed-IC" library_urn="urn:adsk.eagle:library:470" package="SOT-223" package3d_urn="urn:adsk.eagle:package:32638/1" value="CJT1117-5.0-SOT223" x="-6" y="-1" smashed="yes" rot="R180">
+<attribute name="LCSC" value="C89273" x="-6" y="-1" size="1.778" layer="27" rot="R180" display="off"/>
 <attribute name="MPN" value="CJT1117-5.0" x="7" y="30" size="1.778" layer="27" rot="R180" display="off"/>
 <attribute name="VALUE" x="-12.71" y="-6.645" size="0.8128" layer="21"/>
 </element>
-<element name="U$9" library="SparkFun-DiscreteSemi" package="SO08" value="MOSFET-PCHANNEL-SOIC8SOIC8" x="-5" y="17" smashed="yes">
+<element name="U9" library="SparkFun-DiscreteSemi" package="SO08" value="MOSFET-PCHANNEL-SOIC8SOIC8" x="-5" y="17" smashed="yes">
 <attribute name="LCSC" value="C143671" x="-25" y="-5" size="1.778" layer="27" display="off"/>
 <attribute name="VALUE" x="-13.87" y="21.765" size="0.8128" layer="21"/>
@@
 </signal>
 <signal name="VBUS" class="1">
-<contactref element="U$9" pad="1"/>
-<contactref element="U$9" pad="2"/>
-<contactref element="U$9" pad="3"/>
+<contactref element="U9" pad="1"/>
+<contactref element="U9" pad="2"/>
+<contactref element="U9" pad="3"/>
 <contactref element="R7" pad="P$2"/>
 <contactref element="R9" pad="P$2"/>
@@
 <signal name="VOUT">
 <contactref element="U1" pad="3"/>
-<contactref element="U$9" pad="8"/>
-<contactref element="U$9" pad="7"/>
-<contactref element="U$9" pad="6"/>
-<contactref element="U$9" pad="5"/>
+<contactref element="U9" pad="8"/>
+<contactref element="U9" pad="7"/>
+<contactref element="U9" pad="6"/>
+<contactref element="U9" pad="5"/>
 <contactref element="C17" pad="2"/>
 <contactref element="C18" pad="2"/>
@@
 </signal>
 <signal name="GATE">
-<contactref element="U$9" pad="4"/>
+<contactref element="U9" pad="4"/>
 <contactref element="R9" pad="P$1"/>
 <contactref element="R8" pad="P$2"/>
