File: power board/haasoscope_pro_power_board.brd (EAGLE design)
At the start: 72.4 x 97.5 mm, 105 parts, among them IC1 TPS5430DDAR, IC10 TPS5430DDAR, IC11 TPS7A7200RGTR, IC12 TPS7A7200RGTR, IC14 TPS7A7200RGTR, IC2 TPS5430DDAR, IC3 TPS7A7200RGTR, IC4 TPS5430DDAR, IC5 TPS72325DBVR, IC6 TPS5430DDAR, IC7 TPS7A7200RGTR, IC8 TPS5430DDAR, IC9 TPS7A7200RGTR, J1 2p-2.54, J10 2p-2.54, J11 2p-2.54, J12 2p-2.54, J13 2p-2.54, J15 2p-2.54, J2 2p-2.54, J3 2p-2.54, J4 2p-2.54, J5 2p-2.54, J6 2p-2.54, J7 2p-2.54, J8 2p-2.54, J9 2p-2.54

Commit message: power connector etc
Parts:
- added J14: 8pin, SparkFun-Connectors:1X08
Connections:
- net 1V1OUT: now also J14.4
- net 1V9DOUT: now also J14.6
- net 1V9OUT: now also J14.5
- net 2V5DOUT: now also J14.8
- net 3V3OUT: now also J14.1
- net GND: now also J14.2, J14.3, J14.7
Routing:
- net 2V5DOUT: track 20.0 -> 56.6 mm
- net 1V9DOUT: track 16.1 -> 44.8 mm
- net 1V9OUT: track 20.0 -> 44.8 mm
- net 1V1OUT: track 19.9 -> 31.9 mm
- net 3V3OUT: track 26.3 -> 37.5 mm
Other:
- board size 72.4 x 97.5 mm -> 77.5 x 97.5 mm
- board text added: "1.1V"
- board text added: "1.9V"
- board text added: "1.9VD"
- board text added: "2.5VD"
- board text added: "3.3V"
- board text added: "3V3"
- board text removed: "1.1V out GND"
- board text removed: "3.3V out GND"
Changed lines of the file:
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@@
 <drawing>
 <settings>
-<setting alwaysvectorfont="no"/>
+<setting alwaysvectorfont="yes"/>
 <setting verticaltext="up"/>
 </settings>
-<grid distance="50" unitdist="mil" unit="mil" style="lines" multiple="1" display="no" altdistance="5" altunitdist="mil" altunit="mil"/>
+<grid distance="1" unitdist="mm" unit="mm" style="lines" multiple="1" display="no" altdistance="0.1" altunitdist="mm" altunit="mm"/>
 <layers>
 <layer number="1" name="Top" color="12" fill="1" visible="yes" active="yes"/>
@@
 <board>
 <plain>
-<wire x1="1.27" y1="1.27" x2="73.64" y2="1.27" width="0" layer="20"/>
+<wire x1="-3.81" y1="1.27" x2="73.64" y2="1.27" width="0" layer="20"/>
 <wire x1="73.64" y1="1.27" x2="73.64" y2="98.73" width="0" layer="20"/>
-<wire x1="73.64" y1="98.73" x2="1.27" y2="98.73" width="0" layer="20"/>
-<wire x1="1.27" y1="98.73" x2="1.27" y2="1.27" width="0" layer="20"/>
+<wire x1="73.64" y1="98.73" x2="-3.81" y2="98.73" width="0" layer="20"/>
+<wire x1="-3.81" y1="98.73" x2="-3.81" y2="1.27" width="0" layer="20"/>
 <text x="6.477" y="2.921" size="0.8128" layer="21" font="vector">Haasoscope Pro
 Power board, v1.0
 by Dr. Andy Haas</text>
-<hole x="3.81" y="96.52" drill="1.6002"/>
-<hole x="3.81" y="3.81" drill="1.6002"/>
+<hole x="-1.19" y="96.52" drill="1.6002"/>
+<hole x="-1.19" y="3.81" drill="1.6002"/>
 <text x="72.898" y="24.765" size="0.8128" layer="21" rot="R180">2.8V+
 out
@@
 <wire x1="43.18" y1="87.63" x2="41.91" y2="86.36" width="0.1524" layer="21"/>
 <wire x1="41.91" y1="86.36" x2="40.64" y2="87.63" width="0.1524" layer="21"/>
-<text x="5.588" y="93.345" size="0.8128" layer="21" rot="R180">3.3V
-out
-GND</text>
 <text x="5.588" y="62.865" size="0.8128" layer="21" rot="R180">1.9V
 out
 GND</text>
-<text x="5.588" y="78.105" size="0.8128" layer="21" rot="R180">1.1V
-out
-GND</text>
+<text x="9.588" y="73.105" size="0.8128" layer="21" rot="R180">GND</text>
 <text x="4.318" y="29.845" size="0.8128" layer="21" rot="R180">2.5V
 out
@@
 <wire x1="2.54" y1="15.24" x2="20.32" y2="15.24" width="0.3048" layer="21"/>
 <wire x1="20.32" y1="15.24" x2="20.32" y2="2.54" width="0.3048" layer="21"/>
-<wire x1="3.81" y1="82.55" x2="22.86" y2="82.55" width="0.3048" layer="21"/>
+<wire x1="6.81" y1="82.55" x2="22.86" y2="82.55" width="0.3048" layer="21"/>
 <wire x1="22.86" y1="82.55" x2="22.86" y2="45.72" width="0.3048" layer="21"/>
-<wire x1="22.86" y1="45.72" x2="2.54" y2="45.72" width="0.3048" layer="21"/>
+<wire x1="22.86" y1="45.72" x2="6.54" y2="45.72" width="0.3048" layer="21"/>
+<text x="4.5" y="72" size="0.8128" layer="21" rot="R180">2.5VD</text>
+<text x="4.5" y="77.5" size="0.8128" layer="21" rot="R180">1.9VD</text>
+<text x="3.5" y="82.5" size="0.8128" layer="21" rot="R180">1.1V</text>
+<text x="3.5" y="90" size="0.8128" layer="21" rot="R180">3V3</text>
+<text x="3.5" y="87.5" size="0.8128" layer="21" rot="R180">GND</text>
+<text x="3.5" y="85" size="0.8128" layer="21" rot="R180">GND</text>
+<text x="3.5" y="80" size="0.8128" layer="21" rot="R180">1.9V</text>
+<text x="3.5" y="74.5" size="0.8128" layer="21" rot="R180">GND</text>
+<text x="9.588" y="80.105" size="0.8128" layer="21" rot="R180">1.1V</text>
+<text x="8.588" y="88.105" size="0.8128" layer="21" rot="R180">GND</text>
+<text x="8.588" y="96.105" size="0.8128" layer="21" rot="R180">3.3V</text>
 </plain>
 <attributes>
@@
 <element name="C38" library="Nordic_nRF" library_urn="urn:adsk.eagle:library:169009" package="RESC0805_N" package3d_urn="urn:adsk.eagle:package:2593736/1" value="10uF" x="12.7" y="39.37" smashed="yes" rot="R270"/>
 <element name="C43" library="Nordic_nRF" library_urn="urn:adsk.eagle:library:169009" package="RESC0402_N" package3d_urn="urn:adsk.eagle:package:2593732/1" value="0.1uF" x="10.16" y="39.37" smashed="yes" rot="R270"/>
+<element name="J14" library="SparkFun-Connectors" library_urn="urn:adsk.eagle:library:513" package="1X08" package3d_urn="urn:adsk.eagle:package:38138/1" value="8pin" x="-1.27" y="89.71" smashed="yes" rot="R270">
+<attribute name="PROD_ID" value="CONN-08438" x="-1.27" y="89.71" size="1.778" layer="27" rot="R270" display="off"/>
+</element>
 </elements>
 <signals>
 <signal name="GND" airwireshidden="yes">
 <polygon width="0.1524" layer="16">
-<vertex x="0" y="101.6"/>
+<vertex x="-6.35" y="101.6"/>
 <vertex x="74.93" y="101.6"/>
 <vertex x="74.93" y="0"/>
-<vertex x="0" y="0"/>
+<vertex x="-6.35" y="0"/>
 </polygon>
 <contactref element="R2" pad="P$1"/>
@@
 <contactref element="C2" pad="2"/>
 <polygon width="0.1524" layer="1">
-<vertex x="-1.27" y="100.33"/>
+<vertex x="-5.08" y="100.33"/>
 <vertex x="76.2" y="100.33"/>
 <vertex x="76.2" y="-1.27"/>
-<vertex x="-1.27" y="-1.27"/>
+<vertex x="-5.08" y="-1.27"/>
 </polygon>
 <via x="39.751" y="30.48" extent="1-16" drill="0.35"/>
@@
 <wire x1="19.05" y1="39.37" x2="19.3" y2="39.12" width="0.3048" layer="1"/>
 <wire x1="19.3" y1="39.12" x2="20.55" y2="39.12" width="0.3048" layer="1"/>
+<contactref element="J14" pad="2"/>
+<contactref element="J14" pad="7"/>
+<contactref element="J14" pad="3"/>
 </signal>
 <signal name="2V8-">
@@
 <wire x1="10.52" y1="92.35" x2="10.16" y2="91.99" width="0.3048" layer="1"/>
 <wire x1="10.16" y1="91.99" x2="8.34" y2="91.99" width="0.3048" layer="1"/>
-<wire x1="8.34" y1="91.99" x2="7.62" y2="92.71" width="0.3048" layer="1"/>
+<wire x1="8.34" y1="91.99" x2="8.165" y2="92.165" width="0.3048" layer="1"/>
+<wire x1="8.165" y1="92.165" x2="7.62" y2="92.71" width="0.3048" layer="1"/>
 <wire x1="17.55" y1="92.19" x2="18.3" y2="92.94" width="0.3048" layer="1"/>
 <wire x1="18.3" y1="92.94" x2="18.5888" y2="92.94" width="0.3048" layer="1"/>
@@
 <wire x1="16.4597375" y1="91.94" x2="17.3935375" y2="92.8738" width="0.8128" layer="1"/>
 <wire x1="17.3935375" y1="92.8738" x2="18.5226" y2="92.8738" width="0.8128" layer="1"/>
+<contactref element="J14" pad="1"/>
+<wire x1="-1.27" y1="89.71" x2="2" y2="92.98" width="1.27" layer="1"/>
+<wire x1="2" y1="92.98" x2="2" y2="93" width="1.27" layer="1"/>
+<wire x1="2" y1="93" x2="7.33" y2="93" width="1.27" layer="1"/>
+<wire x1="7.33" y1="93" x2="8.165" y2="92.165" width="1.27" layer="1"/>
 </signal>
 <signal name="PG3V3">
@@
 <wire x1="18.3" y1="62.46" x2="18.5888" y2="62.46" width="0.3048" layer="1"/>
 <wire x1="18.5888" y1="62.46" x2="18.8" y2="62.46" width="0.3048" layer="1"/>
-<wire x1="7.62" y1="62.23" x2="10.16" y2="62.23" width="0.8128" layer="1"/>
+<wire x1="7.62" y1="62.23" x2="10" y2="62.23" width="0.8128" layer="1"/>
+<wire x1="10" y1="62.23" x2="10.16" y2="62.23" width="0.8128" layer="1"/>
 <wire x1="10.16" y1="62.23" x2="10.52" y2="61.87" width="0.8128" layer="1"/>
 <wire x1="10.16" y1="61.51" x2="10.71" y2="62.06" width="0.8128" layer="1"/>
@@
 <wire x1="16.462634375" y1="61.462896875" x2="17.3935375" y2="62.3938" width="0.8128" layer="1"/>
 <wire x1="17.3935375" y1="62.3938" x2="18.5226" y2="62.3938" width="0.8128" layer="1"/>
+<contactref element="J14" pad="5"/>
+<wire x1="-1.27" y1="79.55" x2="0.45" y2="79.55" width="1.27" layer="1"/>
+<wire x1="5" y1="75" x2="5" y2="64" width="1.27" layer="1"/>
+<wire x1="5" y1="64" x2="6.77" y2="62.23" width="1.27" layer="1"/>
+<wire x1="6.77" y1="62.23" x2="10" y2="62.23" width="1.27" layer="1"/>
+<wire x1="0.45" y1="79.55" x2="5" y2="75" width="1.27" layer="1"/>
 </signal>
 <signal name="PG1V9">
@@
 <wire x1="10.52" y1="77.11" x2="10.16" y2="76.75" width="0.3048" layer="1"/>
 <wire x1="10.16" y1="76.75" x2="8.34" y2="76.75" width="0.3048" layer="1"/>
-<wire x1="8.34" y1="76.75" x2="7.62" y2="77.47" width="0.3048" layer="1"/>
+<wire x1="8.34" y1="76.75" x2="8.045" y2="77.045" width="0.3048" layer="1"/>
+<wire x1="8.045" y1="77.045" x2="7.62" y2="77.47" width="0.3048" layer="1"/>
 <wire x1="17.55" y1="76.95" x2="18.3" y2="77.7" width="0.3048" layer="1"/>
 <wire x1="18.3" y1="77.7" x2="18.546" y2="77.7" width="0.3048" layer="1"/>
@@
 <wire x1="15.24" y1="76.7" x2="16.24" y2="77.7" width="0.8128" layer="1"/>
 <wire x1="16.24" y1="77.7" x2="18.546" y2="77.7" width="0.8128" layer="1"/>
+<contactref element="J14" pad="4"/>
+<wire x1="-1.27" y1="82.09" x2="3.91" y2="82.09" width="1.27" layer="1"/>
+<wire x1="8.045" y1="77.955" x2="8.045" y2="77.045" width="1.27" layer="1"/>
+<wire x1="3.91" y1="82.09" x2="8.045" y2="77.955" width="1.27" layer="1"/>
 </signal>
 <signal name="PG1V1">
@@
 <wire x1="16.4597375" y1="51.3" x2="17.3935375" y2="52.2338" width="0.8128" layer="1"/>
 <wire x1="17.3935375" y1="52.2338" x2="18.5226" y2="52.2338" width="0.8128" layer="1"/>
+<contactref element="J14" pad="6"/>
+<wire x1="-1.27" y1="77.01" x2="2" y2="73.74" width="1.27" layer="1"/>
+<wire x1="2" y1="57.69" x2="7.62" y2="52.07" width="1.27" layer="1"/>
+<wire x1="2" y1="73.74" x2="2" y2="57.69" width="1.27" layer="1"/>
 </signal>
 <signal name="N$7">
@@
 <wire x1="18.3" y1="40.87" x2="18.5888" y2="40.87" width="0.3048" layer="1"/>
 <wire x1="18.5888" y1="40.87" x2="18.8" y2="40.87" width="0.3048" layer="1"/>
-<wire x1="7.62" y1="40.64" x2="10.16" y2="40.64" width="0.8128" layer="1"/>
+<wire x1="7.62" y1="40.64" x2="8" y2="40.64" width="0.8128" layer="1"/>
+<wire x1="8" y1="40.64" x2="10.16" y2="40.64" width="0.8128" layer="1"/>
 <wire x1="10.16" y1="40.64" x2="10.52" y2="40.28" width="0.8128" layer="1"/>
 <wire x1="10.16" y1="39.92" x2="10.71" y2="40.47" width="0.8128" layer="1"/>
@@
 <wire x1="15.24" y1="39.87" x2="16.24" y2="40.87" width="0.8128" layer="1"/>
 <wire x1="16.24" y1="40.87" x2="18.5888" y2="40.87" width="0.8128" layer="1"/>
+<contactref element="J14" pad="8"/>
+<wire x1="-1.27" y1="71.93" x2="-1.27" y2="47.27" width="1.27" layer="1"/>
+<wire x1="5.36" y1="40.64" x2="8" y2="40.64" width="1.27" layer="1"/>
+<wire x1="-1.27" y1="47.27" x2="5.36" y2="40.64" width="1.27" layer="1"/>
 </signal>
 <signal name="PG2V5D">

Commit message: power connector etc
Parts:
- removed J14: 8pin, SparkFun-Connectors:1X08
- added J16: 8pin, SparkFun-Connectors:1X08
Connections:
- net 1V1OUT: now also J16.2; no longer J14.4
- net 1V9DOUT: now also J16.4; no longer J14.6
- net 1V9OUT: now also J16.3; no longer J14.5
- net 2V5-: now also J16.8
- net 2V5DOUT: now also J16.6; no longer J14.8
- net 2V5OUT: now also J16.7
- net 3V3OUT: now also J16.1; no longer J14.1
- net GND: now also J16.5; no longer J14.2, J14.3, J14.7
Routing:
- net 2V5-: track 6.76 -> 52.7 mm
- net 2V5OUT: track 16.4 -> 52.9 mm
- net 3V3OUT: track 37.5 -> 50.1 mm
- net 1V9OUT: track 44.8 -> 36.0 mm
- net 2V5DOUT: track 56.6 -> 50.2 mm
- net 1V9DOUT: track 44.8 -> 39.3 mm
- net 1V1OUT: track 31.9 -> 30.2 mm
Other:
- board text added: "2v5+"
- board text added: "2v5-"
- board text removed: "1.9V out GND"
Changed lines of the file:
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@@
 <wire x1="43.18" y1="87.63" x2="41.91" y2="86.36" width="0.1524" layer="21"/>
 <wire x1="41.91" y1="86.36" x2="40.64" y2="87.63" width="0.1524" layer="21"/>
-<text x="5.588" y="62.865" size="0.8128" layer="21" rot="R180">1.9V
-out
-GND</text>
+<text x="8.588" y="64.865" size="0.8128" layer="21" rot="R180">1.9V</text>
 <text x="9.588" y="73.105" size="0.8128" layer="21" rot="R180">GND</text>
 <text x="4.318" y="29.845" size="0.8128" layer="21" rot="R180">2.5V
@@
 <wire x1="22.86" y1="82.55" x2="22.86" y2="45.72" width="0.3048" layer="21"/>
 <wire x1="22.86" y1="45.72" x2="6.54" y2="45.72" width="0.3048" layer="21"/>
-<text x="4.5" y="72" size="0.8128" layer="21" rot="R180">2.5VD</text>
-<text x="4.5" y="77.5" size="0.8128" layer="21" rot="R180">1.9VD</text>
-<text x="3.5" y="82.5" size="0.8128" layer="21" rot="R180">1.1V</text>
-<text x="3.5" y="90" size="0.8128" layer="21" rot="R180">3V3</text>
-<text x="3.5" y="87.5" size="0.8128" layer="21" rot="R180">GND</text>
-<text x="3.5" y="85" size="0.8128" layer="21" rot="R180">GND</text>
-<text x="3.5" y="80" size="0.8128" layer="21" rot="R180">1.9V</text>
-<text x="3.5" y="74.5" size="0.8128" layer="21" rot="R180">GND</text>
+<text x="4.3" y="64.8" size="0.8128" layer="21" rot="R180">2.5VD</text>
+<text x="4.2" y="69.5" size="0.8128" layer="21" rot="R180">1.9VD</text>
+<text x="3.5" y="74.5" size="0.8128" layer="21" rot="R180">1.1V</text>
+<text x="3.3" y="77.3" size="0.8128" layer="21" rot="R180">3V3</text>
+<text x="3.5" y="72" size="0.8128" layer="21" rot="R180">1.9V</text>
+<text x="3.5" y="67.2" size="0.8128" layer="21" rot="R180">GND</text>
 <text x="9.588" y="80.105" size="0.8128" layer="21" rot="R180">1.1V</text>
 <text x="8.588" y="88.105" size="0.8128" layer="21" rot="R180">GND</text>
 <text x="8.588" y="96.105" size="0.8128" layer="21" rot="R180">3.3V</text>
+<text x="3.7" y="61.9" size="0.8128" layer="21" rot="R180">2v5+</text>
+<text x="3.6" y="59.9" size="0.8128" layer="21" rot="R180">2v5-</text>
+<text x="9.588" y="58.105" size="0.8128" layer="21" rot="R180">GND</text>
 </plain>
 <attributes>
@@
 <element name="C38" library="Nordic_nRF" library_urn="urn:adsk.eagle:library:169009" package="RESC0805_N" package3d_urn="urn:adsk.eagle:package:2593736/1" value="10uF" x="12.7" y="39.37" smashed="yes" rot="R270"/>
 <element name="C43" library="Nordic_nRF" library_urn="urn:adsk.eagle:library:169009" package="RESC0402_N" package3d_urn="urn:adsk.eagle:package:2593732/1" value="0.1uF" x="10.16" y="39.37" smashed="yes" rot="R270"/>
-<element name="J14" library="SparkFun-Connectors" library_urn="urn:adsk.eagle:library:513" package="1X08" package3d_urn="urn:adsk.eagle:package:38138/1" value="8pin" x="-1.27" y="89.71" smashed="yes" rot="R270">
-<attribute name="PROD_ID" value="CONN-08438" x="-1.27" y="89.71" size="1.778" layer="27" rot="R270" display="off"/>
+<element name="J16" library="SparkFun-Connectors" library_urn="urn:adsk.eagle:library:513" package="1X08" package3d_urn="urn:adsk.eagle:package:38138/1" value="8pin" x="-1" y="77" smashed="yes" rot="R270">
+<attribute name="PROD_ID" value="CONN-08438" x="-1" y="77" size="1.778" layer="27" rot="R270" display="off"/>
 </element>
 </elements>
@@
 <wire x1="19.05" y1="39.37" x2="19.3" y2="39.12" width="0.3048" layer="1"/>
 <wire x1="19.3" y1="39.12" x2="20.55" y2="39.12" width="0.3048" layer="1"/>
-<contactref element="J14" pad="2"/>
-<contactref element="J14" pad="7"/>
-<contactref element="J14" pad="3"/>
+<contactref element="J16" pad="5"/>
 </signal>
 <signal name="2V8-">
@@
 <wire x1="16.4597375" y1="91.94" x2="17.3935375" y2="92.8738" width="0.8128" layer="1"/>
 <wire x1="17.3935375" y1="92.8738" x2="18.5226" y2="92.8738" width="0.8128" layer="1"/>
-<contactref element="J14" pad="1"/>
-<wire x1="-1.27" y1="89.71" x2="2" y2="92.98" width="1.27" layer="1"/>
-<wire x1="2" y1="92.98" x2="2" y2="93" width="1.27" layer="1"/>
 <wire x1="2" y1="93" x2="7.33" y2="93" width="1.27" layer="1"/>
 <wire x1="7.33" y1="93" x2="8.165" y2="92.165" width="1.27" layer="1"/>
+<contactref element="J16" pad="1"/>
+<wire x1="2" y1="93" x2="-1" y2="90" width="1.27" layer="1"/>
+<wire x1="-1" y1="90" x2="-1" y2="77" width="1.27" layer="1"/>
 </signal>
 <signal name="PG3V3">
@@
 <wire x1="10.52" y1="61.87" x2="10.16" y2="61.51" width="0.3048" layer="1"/>
 <wire x1="10.16" y1="61.51" x2="8.34" y2="61.51" width="0.3048" layer="1"/>
-<wire x1="8.34" y1="61.51" x2="7.62" y2="62.23" width="0.3048" layer="1"/>
+<wire x1="8.34" y1="61.51" x2="7.925" y2="61.925" width="0.3048" layer="1"/>
+<wire x1="7.925" y1="61.925" x2="7.62" y2="62.23" width="0.3048" layer="1"/>
 <wire x1="17.55" y1="61.71" x2="18.3" y2="62.46" width="0.3048" layer="1"/>
 <wire x1="18.3" y1="62.46" x2="18.5888" y2="62.46" width="0.3048" layer="1"/>
@@
 <wire x1="16.462634375" y1="61.462896875" x2="17.3935375" y2="62.3938" width="0.8128" layer="1"/>
 <wire x1="17.3935375" y1="62.3938" x2="18.5226" y2="62.3938" width="0.8128" layer="1"/>
-<contactref element="J14" pad="5"/>
-<wire x1="-1.27" y1="79.55" x2="0.45" y2="79.55" width="1.27" layer="1"/>
-<wire x1="5" y1="75" x2="5" y2="64" width="1.27" layer="1"/>
-<wire x1="5" y1="64" x2="6.77" y2="62.23" width="1.27" layer="1"/>
-<wire x1="6.77" y1="62.23" x2="10" y2="62.23" width="1.27" layer="1"/>
-<wire x1="0.45" y1="79.55" x2="5" y2="75" width="1.27" layer="1"/>
+<contactref element="J16" pad="3"/>
+<wire x1="-1" y1="71.92" x2="3.08" y2="71.92" width="1.27" layer="1"/>
+<wire x1="7.925" y1="67.075" x2="7.925" y2="61.925" width="1.27" layer="1"/>
+<wire x1="3.08" y1="71.92" x2="7.925" y2="67.075" width="1.27" layer="1"/>
 </signal>
 <signal name="PG1V9">
@@
 <wire x1="18.3" y1="77.7" x2="18.546" y2="77.7" width="0.3048" layer="1"/>
 <wire x1="18.546" y1="77.7" x2="18.8" y2="77.7" width="0.3048" layer="1"/>
-<wire x1="7.62" y1="77.47" x2="10.16" y2="77.47" width="0.8128" layer="1"/>
+<wire x1="7.62" y1="77.47" x2="8" y2="77.47" width="0.8128" layer="1"/>
+<wire x1="8" y1="77.47" x2="10.16" y2="77.47" width="0.8128" layer="1"/>
 <wire x1="10.16" y1="77.47" x2="10.52" y2="77.11" width="0.8128" layer="1"/>
 <wire x1="10.16" y1="76.75" x2="10.71" y2="77.3" width="0.8128" layer="1"/>
@@
 <wire x1="15.24" y1="76.7" x2="16.24" y2="77.7" width="0.8128" layer="1"/>
 <wire x1="16.24" y1="77.7" x2="18.546" y2="77.7" width="0.8128" layer="1"/>
-<contactref element="J14" pad="4"/>
-<wire x1="-1.27" y1="82.09" x2="3.91" y2="82.09" width="1.27" layer="1"/>
-<wire x1="8.045" y1="77.955" x2="8.045" y2="77.045" width="1.27" layer="1"/>
-<wire x1="3.91" y1="82.09" x2="8.045" y2="77.955" width="1.27" layer="1"/>
+<contactref element="J16" pad="2"/>
+<wire x1="-1" y1="74.46" x2="2.01" y2="77.47" width="1.27" layer="1"/>
+<wire x1="2.01" y1="77.47" x2="8" y2="77.47" width="1.27" layer="1"/>
 </signal>
 <signal name="PG1V1">
@@
 <wire x1="11.43" y1="19.515" x2="13.845" y2="19.515" width="0.8128" layer="1"/>
 <wire x1="13.845" y1="19.515" x2="13.99" y2="19.37" width="0.8128" layer="1"/>
+<contactref element="J16" pad="8"/>
+<wire x1="-1" y1="59.22" x2="-1" y2="23" width="1.27" layer="1"/>
+<wire x1="1.68" y1="20.32" x2="7.62" y2="20.32" width="1.27" layer="1"/>
+<wire x1="-1" y1="23" x2="1.68" y2="20.32" width="1.27" layer="1"/>
 </signal>
 <signal name="N$4">
@@
 <wire x1="15.5747375" y1="28.825" x2="16.1235375" y2="29.3738" width="0.8128" layer="1"/>
 <wire x1="16.1235375" y1="29.3738" x2="17.2526" y2="29.3738" width="0.8128" layer="1"/>
+<contactref element="J16" pad="7"/>
+<wire x1="-1" y1="61.76" x2="1" y2="59.76" width="1.27" layer="1"/>
+<wire x1="4.79" y1="29.21" x2="6.35" y2="29.21" width="1.27" layer="1"/>
+<wire x1="1" y1="59.76" x2="1" y2="33" width="1.27" layer="1"/>
+<wire x1="1" y1="33" x2="4.79" y2="29.21" width="1.27" layer="1"/>
 </signal>
 <signal name="PG25">
@@
 <wire x1="18.3" y1="52.3" x2="18.5888" y2="52.3" width="0.3048" layer="1"/>
 <wire x1="18.5888" y1="52.3" x2="18.8" y2="52.3" width="0.3048" layer="1"/>
-<wire x1="7.62" y1="52.07" x2="9.44" y2="52.07" width="0.8128" layer="1"/>
+<wire x1="7.62" y1="52.07" x2="8" y2="52.07" width="0.8128" layer="1"/>
+<wire x1="8" y1="52.07" x2="9.44" y2="52.07" width="0.8128" layer="1"/>
 <wire x1="9.44" y1="52.07" x2="10.16" y2="51.35" width="0.8128" layer="1"/>
 <wire x1="10.16" y1="51.35" x2="10.71" y2="51.9" width="0.8128" layer="1"/>
@@
 <wire x1="16.4597375" y1="51.3" x2="17.3935375" y2="52.2338" width="0.8128" layer="1"/>
 <wire x1="17.3935375" y1="52.2338" x2="18.5226" y2="52.2338" width="0.8128" layer="1"/>
-<contactref element="J14" pad="6"/>
-<wire x1="-1.27" y1="77.01" x2="2" y2="73.74" width="1.27" layer="1"/>
-<wire x1="2" y1="57.69" x2="7.62" y2="52.07" width="1.27" layer="1"/>
-<wire x1="2" y1="73.74" x2="2" y2="57.69" width="1.27" layer="1"/>
+<contactref element="J16" pad="4"/>
+<wire x1="-1" y1="69.38" x2="2.62" y2="69.38" width="1.27" layer="1"/>
+<wire x1="2.62" y1="69.38" x2="5" y2="67" width="1.27" layer="1"/>
+<wire x1="5" y1="67" x2="5" y2="55" width="1.27" layer="1"/>
+<wire x1="5" y1="55" x2="7.93" y2="52.07" width="1.27" layer="1"/>
+<wire x1="7.93" y1="52.07" x2="8" y2="52.07" width="1.27" layer="1"/>
 </signal>
 <signal name="N$7">
@@
 <wire x1="15.24" y1="39.87" x2="16.24" y2="40.87" width="0.8128" layer="1"/>
 <wire x1="16.24" y1="40.87" x2="18.5888" y2="40.87" width="0.8128" layer="1"/>
-<contactref element="J14" pad="8"/>
-<wire x1="-1.27" y1="71.93" x2="-1.27" y2="47.27" width="1.27" layer="1"/>
 <wire x1="5.36" y1="40.64" x2="8" y2="40.64" width="1.27" layer="1"/>
-<wire x1="-1.27" y1="47.27" x2="5.36" y2="40.64" width="1.27" layer="1"/>
+<contactref element="J16" pad="6"/>
+<wire x1="-1" y1="64.3" x2="1.2776" y2="64.3" width="1.27" layer="1"/>
+<wire x1="1.2776" y1="64.3" x2="3.1776" y2="62.4" width="1.27" layer="1"/>
+<wire x1="3.1776" y1="62.4" x2="3.1776" y2="42.8224" width="1.27" layer="1"/>
+<wire x1="3.1776" y1="42.8224" x2="5.36" y2="40.64" width="1.27" layer="1"/>
 </signal>
 <signal name="PG2V5D">

Commit message: minor
Other:
- board text added: "12V in"
- board text removed: "Vin"
Changed lines of the file:
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@@
 <text x="59.817" y="12.446" size="0.8128" layer="21" rot="R180">+</text>
 <text x="4.953" y="6.223" size="0.8128" layer="21" rot="R180">GND</text>
-<text x="4.572" y="13.589" size="0.8128" layer="21" rot="R180">Vin</text>
+<text x="4.572" y="13.589" size="0.8128" layer="21" rot="R180">12V in</text>
 <wire x1="38.1" y1="22.86" x2="40.64" y2="22.86" width="0.1524" layer="21"/>
 <wire x1="40.64" y1="22.86" x2="39.37" y2="21.59" width="0.1524" layer="21"/>
