File: power board/haasoscope_pro_power_board - 5V.brd (EAGLE design)
At the start: 77.5 x 97.5 mm, 123 parts, among them CN1 12Vin, IC11 TPS7A7200RGTR, IC12 TPS7A7200RGTR, IC14 TPS7A7200RGTR, IC3 TPS7A7200RGTR, IC5 TPS72325DBVR, IC7 TPS7A7200RGTR, IC9 TPS7A7200RGTR, J1 2p-2.54, J10 2p-2.54, J11 2p-2.54, J12 2p-2.54, J13 2p-2.54, J14 2p-2.54, J15 2p-2.54, J16 8pin, J17 2p-2.54, J18 2p-2.54, J19 2p-2.54, J2 2p-2.54, J20 2p-2.54, J3 2p-2.54, J4 2p-2.54, J5 2p-2.54, J6 2p-2.54, J7 2p-2.54, J8 2p-2.54, J9 2p-2.54

Commit message: add diode
Parts:
- added D6: B340A, SparkFun-DiscreteSemi:SMA-DIODE
- moved J1 59.0 mm to (6.00, 4.00)
- moved R1 3.81 mm to (70.9, 9.70), turned to 90 degrees
- moved C52 1.10 mm to (61.9, 16.9), turned to 180 degrees
Connections:
- net 2V8-: now also D6.A
- net GND: now also D6.C
Routing:
- net 5V: track 216.7 -> 260.3 mm
- net 2V8-: track 83.3 -> 92.7 mm
- net GND: track 140.4 -> 146.7 mm
Other:
- board text added: "12V"
Changed lines of the file:
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@@
 <text x="69.004" y="24.917" size="0.8128" layer="21" rot="R270">-</text>
 <text x="62.654" y="24.917" size="0.8128" layer="21" rot="R270">+</text>
-<text x="61.111" y="5.572" size="0.8128" layer="21" rot="R270">5V in</text>
-<text x="68.777" y="4.953" size="0.8128" layer="21" rot="R270">GND</text>
-<text x="71.777" y="17.953" size="0.8128" layer="21" rot="R270">GND</text>
-<text x="66.428" y="14.111" size="0.8128" layer="21">5V</text>
+<text x="2.111" y="5.572" size="0.8128" layer="21" rot="R270">5V in</text>
+<text x="9.777" y="4.953" size="0.8128" layer="21" rot="R270">GND</text>
+<text x="71.277" y="17.953" size="0.8128" layer="21" rot="R270">GND</text>
+<text x="64.889" y="16.428" size="0.8128" layer="21" rot="R90">5V</text>
+<wire x1="12.1" y1="9.45" x2="9.56" y2="9.45" width="0.1524" layer="21"/>
+<wire x1="9.56" y1="9.45" x2="10.83" y2="10.72" width="0.1524" layer="21"/>
+<wire x1="10.83" y1="10.72" x2="12.1" y2="9.45" width="0.1524" layer="21"/>
+<wire x1="12.1" y1="10.72" x2="8.29" y2="10.72" width="0.1524" layer="21"/>
+<wire x1="9.56" y1="9.45" x2="7.02" y2="9.45" width="0.1524" layer="21"/>
+<wire x1="8.29" y1="10.72" x2="7.02" y2="10.72" width="0.1524" layer="21"/>
+<wire x1="7.02" y1="9.45" x2="8.29" y2="10.72" width="0.1524" layer="21"/>
+<wire x1="8.29" y1="10.72" x2="9.56" y2="9.45" width="0.1524" layer="21"/>
+<text x="68.428" y="11.711" size="0.8128" layer="21">5V</text>
+<text x="68.428" y="93.511" size="0.8128" layer="21">12V</text>
 </plain>
 <attributes>
@@
 <attribute name="VALUE" x="61.08" y="20.095" size="0.8128" layer="21" rot="R90"/>
 </element>
-<element name="C52" library="Nordic_nRF" library_urn="urn:adsk.eagle:library:169009" package="RESC0402_N" package3d_urn="urn:adsk.eagle:package:2593732/1" value="0.1uF" x="63" y="17" smashed="yes">
-<attribute name="VALUE" x="62.3" y="15" size="0.8128" layer="21"/>
+<element name="C52" library="Nordic_nRF" library_urn="urn:adsk.eagle:library:169009" package="RESC0402_N" package3d_urn="urn:adsk.eagle:package:2593732/1" value="0.1uF" x="61.9" y="16.9" smashed="yes" rot="R180">
+<attribute name="VALUE" x="62.6" y="18.9" size="0.8128" layer="21" rot="R180"/>
 </element>
 <element name="J11" library="Seeed-Connector" library_urn="urn:adsk.eagle:library:478" package="H2-2.54" package3d_urn="urn:adsk.eagle:package:33132/1" value="2p-2.54" x="68" y="17" smashed="yes" rot="R90">
@@
 <attribute name="VALUE" x="65.5" y="49.27" size="0.8128" layer="21" font="vector" rot="R270"/>
 </element>
-<element name="J1" library="Seeed-Connector" library_urn="urn:adsk.eagle:library:478" package="H2-2.54" package3d_urn="urn:adsk.eagle:package:33132/1" value="2p-2.54" x="65" y="4" smashed="yes" rot="R270">
-<attribute name="MPN" value="P125-1102A0BS116A1" x="72" y="4" size="0.8128" layer="27" rot="R270" display="off"/>
+<element name="J1" library="Seeed-Connector" library_urn="urn:adsk.eagle:library:478" package="H2-2.54" package3d_urn="urn:adsk.eagle:package:33132/1" value="2p-2.54" x="6" y="4" smashed="yes" rot="R270">
+<attribute name="MPN" value="P125-1102A0BS116A1" x="13" y="4" size="0.8128" layer="27" rot="R270" display="off"/>
 </element>
 <element name="C1" library="Nordic_nRF" library_urn="urn:adsk.eagle:library:169009" package="RESC0805_N" package3d_urn="urn:adsk.eagle:package:2593736/1" value="10uF" x="66" y="9" smashed="yes" rot="R90"/>
@@
 <attribute name="URL" value="" x="62" y="9" size="0.8128" layer="27" rot="R270" display="off"/>
 </element>
-<element name="R1" library="FlashPCB_Resistors" package="RES-0402" value="3.3k" x="69" y="13" smashed="yes" rot="R270"/>
+<element name="R1" library="FlashPCB_Resistors" package="RES-0402" value="3.3k" x="70.9" y="9.7" smashed="yes" rot="R90"/>
 <element name="C4" library="Nordic_nRF" library_urn="urn:adsk.eagle:library:169009" package="RESC0805_N" package3d_urn="urn:adsk.eagle:package:2593736/1" value="10uF" x="46" y="6" smashed="yes" rot="R180">
 <attribute name="VALUE" x="47" y="8.5" size="0.8128" layer="21" rot="R180"/>
+</element>
+<element name="D6" library="SparkFun-DiscreteSemi" library_urn="urn:adsk.eagle:library:514" package="SMA-DIODE" package3d_urn="urn:adsk.eagle:package:38443/1" value="B340A" x="11" y="10" smashed="yes" rot="R90">
+<attribute name="LCSC" value="C64982" x="11" y="10" size="0.8128" layer="27" rot="R90" display="off"/>
+<attribute name="PROD_ID" value="DIO-09886" x="11" y="10" size="0.8128" layer="27" rot="R90" display="off"/>
+<attribute name="VALUE" x="12.651" y="10" size="0.8128" layer="21" font="vector" rot="R90" align="top-center"/>
 </element>
 </elements>
@@
 <wire x1="60" y1="45.55" x2="60" y2="47" width="0.3048" layer="1"/>
 <via x="60" y="47" extent="1-16" drill="0.35"/>
-<wire x1="63.55" y1="17" x2="64.6" y2="17" width="0.3048" layer="1"/>
-<via x="64.6" y="17" extent="1-16" drill="0.35"/>
+<wire x1="61.35" y1="16.9" x2="59.603078125" y2="16.9" width="0.3048" layer="1"/>
+<wire x1="59.603078125" y1="16.9" x2="59.6" y2="17" width="0.3048" layer="1"/>
+<via x="59.6" y="17" extent="1-16" drill="0.35"/>
 <contactref element="J1" pad="1"/>
 <contactref element="C2" pad="2"/>
@@
 <wire x1="19.25" y1="91.25" x2="19.05" y2="91.44" width="0.3048" layer="1"/>
 <wire x1="20.5" y1="90.75" x2="20.55" y2="90.69" width="0.3048" layer="1"/>
+<contactref element="D6" pad="C"/>
+<wire x1="11" y1="12.15" x2="8.695" y2="12.15" width="1.27" layer="1"/>
+<wire x1="8.695" y1="12.15" x2="6.43" y2="14.415" width="1.27" layer="1"/>
 </signal>
 <signal name="2V8-">
@@
 <wire x1="11.5" y1="17.25" x2="11.49" y2="17.32" width="0.3048" layer="1"/>
 <wire x1="12" y1="17.25" x2="12.55355" y2="17.32" width="0.3048" layer="1"/>
+<contactref element="D6" pad="A"/>
+<wire x1="20" y1="8.73" x2="11.88" y2="8.73" width="1.27" layer="1"/>
+<wire x1="11.88" y1="8.73" x2="11" y2="7.85" width="1.27" layer="1"/>
 </signal>
 <signal name="2V8+">
@@
 <wire x1="65" y1="28.1" x2="65" y2="24.048" width="1.27" layer="1"/>
 <wire x1="65" y1="24.048" x2="62.952" y2="22" width="1.27" layer="1"/>
-<wire x1="62.4626" y1="17.62615" x2="62.4626" y2="17.0126" width="1.27" layer="1"/>
-<wire x1="62.4626" y1="17.0126" x2="62.45" y2="17" width="1.27" layer="1"/>
 <wire x1="62.952" y1="22" x2="62.952" y2="19" width="1.27" layer="1"/>
-<wire x1="62.952" y1="19" x2="62.952" y2="18.11555" width="1.27" layer="1"/>
-<wire x1="62.952" y1="18.11555" x2="62.4626" y2="17.62615" width="1.27" layer="1"/>
+<wire x1="62.952" y1="18.11555" x2="62.952" y2="19" width="1.27" layer="1"/>
 <wire x1="66.73" y1="17" x2="64.73" y2="19" width="1.27" layer="1"/>
 <wire x1="64.73" y1="19" x2="62.952" y2="19" width="1.27" layer="1"/>
-<wire x1="62.45" y1="17" x2="62.45" y2="13.35355" width="1.27" layer="1"/>
 <wire x1="63" y1="48.5" x2="63" y2="50" width="0.3048" layer="1"/>
 <via x="63" y="50" extent="1-16" drill="0.35"/>
@@
 <wire x1="51.28321875" y1="7.5776" x2="51.12271875" y2="7.7381" width="1.27" layer="1"/>
 <wire x1="51.12271875" y1="7.7381" x2="49.55615" y2="7.7381" width="1.27" layer="1"/>
-<wire x1="62.45" y1="13.35355" x2="56.67405" y2="7.5776" width="1.27" layer="1"/>
+<wire x1="56.67405" y1="7.5776" x2="62.45" y2="13.35355" width="1.27" layer="1"/>
 <wire x1="56.67405" y1="7.5776" x2="51.28321875" y2="7.5776" width="1.27" layer="1"/>
-<wire x1="63.73" y1="4" x2="64.6571" y2="4.9271" width="1.27" layer="1"/>
-<wire x1="64.6571" y1="4.9271" x2="64.6571" y2="5.15165" width="1.27" layer="1"/>
 <wire x1="66" y1="6.49455" x2="66" y2="7.9" width="1.27" layer="1"/>
-<wire x1="66" y1="7.9" x2="66" y2="8" width="1.27" layer="1"/>
-<wire x1="66" y1="8" x2="66" y2="8.6126" width="1.27" layer="1"/>
-<wire x1="64.6571" y1="5.15165" x2="66" y2="6.49455" width="1.27" layer="1"/>
+<wire x1="66" y1="7.9" x2="66" y2="8.6126" width="1.27" layer="1"/>
 <wire x1="66" y1="8.6126" x2="68.1374" y2="8.6126" width="1.27" layer="1"/>
 <wire x1="68.1374" y1="8.6126" x2="69" y2="7.75" width="1.27" layer="1"/>
-<wire x1="63.73" y1="4" x2="60.1524" y2="7.5776" width="1.27" layer="1"/>
-<wire x1="60.1524" y1="7.5776" x2="56.67405" y2="7.5776" width="1.27" layer="1"/>
 <wire x1="49.55615" y1="21.7381" x2="62.6901" y2="21.7381" width="1.27" layer="1"/>
 <wire x1="62.6901" y1="21.7381" x2="62.952" y2="22" width="1.27" layer="1"/>
@@
 <wire x1="60" y1="78" x2="60" y2="65.6688" width="1.27" layer="1"/>
 <wire x1="60" y1="65.6688" x2="59.1656" y2="64.8344" width="1.27" layer="1"/>
+<wire x1="65.98195" y1="6.5126" x2="66" y2="6.49455" width="1.27" layer="1"/>
+<wire x1="61.53385" y1="7.5776" x2="62.59885" y2="6.5126" width="1.27" layer="1"/>
+<wire x1="62.59885" y1="6.5126" x2="65.98195" y2="6.5126" width="1.27" layer="1"/>
+<wire x1="56.67405" y1="7.5776" x2="61.53385" y2="7.5776" width="1.27" layer="1"/>
+<wire x1="5.6571" y1="5.15165" x2="6.11835" y2="5.6129" width="1.27" layer="1"/>
+<wire x1="6.11835" y1="5.6129" x2="8.42165" y2="5.6129" width="1.27" layer="1"/>
+<wire x1="4.73" y1="4" x2="5.6571" y2="4.9271" width="1.27" layer="1"/>
+<wire x1="5.6571" y1="4.9271" x2="5.6571" y2="5.15165" width="1.27" layer="1"/>
+<wire x1="10.03455" y1="4" x2="47" y2="4" width="1.27" layer="1"/>
+<wire x1="8.42165" y1="5.6129" x2="10.03455" y2="4" width="1.27" layer="1"/>
+<wire x1="47" y1="4" x2="47.1" y2="4.1" width="1.27" layer="1"/>
+<wire x1="47.1" y1="4.1" x2="47.1" y2="6" width="1.27" layer="1"/>
+<wire x1="62.45" y1="13.35355" x2="62.45" y2="16.9" width="1.27" layer="1"/>
+<wire x1="62.45" y1="16.9" x2="62.45" y2="17.61355" width="1.27" layer="1"/>
+<wire x1="62.45" y1="17.61355" x2="62.952" y2="18.11555" width="1.27" layer="1"/>
 </signal>
 <signal name="N$11">
@@
 <contactref element="D1" pad="CATHODE"/>
 <contactref element="R1" pad="P$2"/>
-<wire x1="69" y1="10.25" x2="69" y2="12.5" width="0.3048" layer="1"/>
+<wire x1="69" y1="10.25" x2="70.9" y2="10.2" width="0.3048" layer="1"/>
+</signal>
+<signal name="SW4">
 </signal>
 </signals>

Commit message: use more standard resistor values
Parts:
- added R2: 15k, FlashPCB_Resistors:RES-0402
- R11, R13, R20: value 55k -> 56k
- R16: value 25k -> 10k
- R25: value 37k -> 39k
- R7: value 71k -> 68k
Connections:
- new net N$14: R16.P$1, R2.P$2
- net GND: now also R2.P$1; no longer R16.P$1
Routing:
- net GND: track 146.7 -> 145.2 mm, vias 50 -> 49
- net N$14: track 0.00 -> 1.00 mm
Changed lines of the file:
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@@
 <attribute name="VALUE" x="57.27" y="93.5" size="0.8128" layer="21" font="vector" rot="R180"/>
 </element>
-<element name="R25" library="FlashPCB_Resistors" package="RES-0402" value="37k" x="56" y="90" smashed="yes" rot="R180">
+<element name="R25" library="FlashPCB_Resistors" package="RES-0402" value="39k" x="56" y="90" smashed="yes" rot="R180">
 <attribute name="VALUE" x="57.27" y="89.5" size="0.8128" layer="21" font="vector" rot="R180"/>
 </element>
@@
 <attribute name="VALUE" x="57.27" y="63.5" size="0.8128" layer="21" font="vector" rot="R180"/>
 </element>
-<element name="R7" library="FlashPCB_Resistors" package="RES-0402" value="71k" x="56" y="60" smashed="yes" rot="R180">
+<element name="R7" library="FlashPCB_Resistors" package="RES-0402" value="68k" x="56" y="60" smashed="yes" rot="R180">
 <attribute name="VALUE" x="57.27" y="59.5" size="0.8128" layer="21" font="vector" rot="R180"/>
 </element>
@@
 <attribute name="VALUE" x="52.27" y="44.5" size="0.8128" layer="21" font="vector" rot="R180"/>
 </element>
-<element name="R11" library="FlashPCB_Resistors" package="RES-0402" value="55k" x="51" y="41" smashed="yes" rot="R180">
+<element name="R11" library="FlashPCB_Resistors" package="RES-0402" value="56k" x="51" y="41" smashed="yes" rot="R180">
 <attribute name="VALUE" x="52.27" y="40.5" size="0.8128" layer="21" font="vector" rot="R180"/>
 </element>
@@
 <attribute name="VALUE" x="52.27" y="30.5" size="0.8128" layer="21" font="vector" rot="R180"/>
 </element>
-<element name="R13" library="FlashPCB_Resistors" package="RES-0402" value="55k" x="51" y="27" smashed="yes" rot="R180">
+<element name="R13" library="FlashPCB_Resistors" package="RES-0402" value="56k" x="51" y="27" smashed="yes" rot="R180">
 <attribute name="VALUE" x="52.27" y="26.5" size="0.8128" layer="21" font="vector" rot="R180"/>
 </element>
@@
 <attribute name="VALUE" x="52.27" y="16.5" size="0.8128" layer="21" font="vector" rot="R180"/>
 </element>
-<element name="R20" library="FlashPCB_Resistors" package="RES-0402" value="55k" x="51" y="13" smashed="yes" rot="R180">
+<element name="R20" library="FlashPCB_Resistors" package="RES-0402" value="56k" x="51" y="13" smashed="yes" rot="R180">
 <attribute name="VALUE" x="52.27" y="12.5" size="0.8128" layer="21" font="vector" rot="R180"/>
 </element>
@@
 </element>
 <element name="C48" library="Nordic_nRF" library_urn="urn:adsk.eagle:library:169009" package="RESC0402_N" package3d_urn="urn:adsk.eagle:package:2593732/1" value="0.1uF" x="69" y="48" smashed="yes" rot="R90">
+<attribute name="LCSC" value="
+C307331" x="69" y="48" size="1.778" layer="27" rot="R90" display="off"/>
 <attribute name="VALUE" x="68" y="47.3" size="0.8128" layer="21" rot="R90"/>
 </element>
@@
 <attribute name="VALUE" x="61.5" y="49.27" size="0.8128" layer="21" font="vector" rot="R270"/>
 </element>
-<element name="R16" library="FlashPCB_Resistors" package="RES-0402" value="25k" x="65" y="48" smashed="yes" rot="R270">
+<element name="R16" library="FlashPCB_Resistors" package="RES-0402" value="10k" x="65" y="48" smashed="yes" rot="R270">
 <attribute name="VALUE" x="65.5" y="49.27" size="0.8128" layer="21" font="vector" rot="R270"/>
 </element>
@@
 <attribute name="PROD_ID" value="DIO-09886" x="11" y="10" size="0.8128" layer="27" rot="R90" display="off"/>
 <attribute name="VALUE" x="12.651" y="10" size="0.8128" layer="21" font="vector" rot="R90" align="top-center"/>
+</element>
+<element name="R2" library="FlashPCB_Resistors" package="RES-0402" value="15k" x="65" y="50" smashed="yes" rot="R270">
+<attribute name="VALUE" x="65.5" y="51.27" size="0.8128" layer="27" font="vector" rot="R270"/>
 </element>
 </elements>
@@
 <contactref element="J11" pad="2"/>
 <contactref element="C51" pad="-"/>
-<contactref element="R16" pad="P$1"/>
 <contactref element="PS7" pad="9"/>
 <wire x1="69.27" y1="17" x2="69" y2="17.27" width="1.27" layer="1"/>
 <wire x1="69" y1="17.27" x2="69" y2="22" width="1.27" layer="1"/>
 <wire x1="69" y1="22" x2="69.048" y2="22" width="1.27" layer="1"/>
-<wire x1="65" y1="48.5" x2="65" y2="50" width="0.3048" layer="1"/>
-<via x="65" y="50" extent="1-16" drill="0.35"/>
 <wire x1="69" y1="48.55" x2="69" y2="50" width="0.3048" layer="1"/>
 <via x="69" y="50" extent="1-16" drill="0.35"/>
@@
 <wire x1="11" y1="12.15" x2="8.695" y2="12.15" width="1.27" layer="1"/>
 <wire x1="8.695" y1="12.15" x2="6.43" y2="14.415" width="1.27" layer="1"/>
+<contactref element="R2" pad="P$1"/>
 </signal>
 <signal name="2V8-">
@@
 <signal name="SW4">
 </signal>
+<signal name="N$14">
+<contactref element="R16" pad="P$1"/>
+<contactref element="R2" pad="P$2"/>
+<wire x1="65" y1="48.5" x2="65" y2="49.5" width="0.3048" layer="1"/>
+</signal>
 </signals>

Commit message: add another 12V cap
Parts:
- added C5: 0.1uF, Nordic_nRF:RESC0402_N
Connections:
- new net N$40: C48.2, C5.1
- net GND: now also C5.2; no longer C48.2
Routing:
- net GND: track 145.2 -> 143.8 mm, vias 49 -> 48
- net N$40: track 0.00 -> 1.30 mm
Changed lines of the file:
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@@
 <attribute name="VALUE" x="65.5" y="51.27" size="0.8128" layer="27" font="vector" rot="R270"/>
+</element>
+<element name="C5" library="Nordic_nRF" library_urn="urn:adsk.eagle:library:169009" package="RESC0402_N" package3d_urn="urn:adsk.eagle:package:2593732/1" value="0.1uF" x="69" y="50.4" smashed="yes" rot="R90">
+<attribute name="LCSC" value="
+C307331" x="69" y="50.4" size="0.8128" layer="27" rot="R90" display="off"/>
 </element>
 </elements>
@@
 <wire x1="20" y1="28.45" x2="20" y2="27.4" width="0.3048" layer="1"/>
 <via x="20" y="27.4" extent="1-16" drill="0.35"/>
-<contactref element="C48" pad="2"/>
-<contactref element="PS7" pad="1"/>
 <contactref element="C50" pad="2"/>
 <contactref element="C52" pad="2"/>
@@
 <wire x1="69" y1="17.27" x2="69" y2="22" width="1.27" layer="1"/>
 <wire x1="69" y1="22" x2="69.048" y2="22" width="1.27" layer="1"/>
-<wire x1="69" y1="48.55" x2="69" y2="50" width="0.3048" layer="1"/>
-<via x="69" y="50" extent="1-16" drill="0.35"/>
 <wire x1="69.048" y1="22" x2="67" y2="22" width="0.3048" layer="1"/>
 <via x="67" y="22" extent="1-16" drill="0.35"/>
-<wire x1="68.712" y1="42.095" x2="69" y2="41.807" width="0.3048" layer="1"/>
-<wire x1="69" y1="41.807" x2="69" y2="41" width="0.3048" layer="1"/>
-<via x="69" y="41" extent="1-16" drill="0.35"/>
 <wire x1="66.1" y1="46.1" x2="66.1" y2="44.1" width="0.3048" layer="1"/>
 <wire x1="66" y1="44" x2="66.1" y2="44.1" width="0.3048" layer="1"/>
@@
 <wire x1="8.695" y1="12.15" x2="6.43" y2="14.415" width="1.27" layer="1"/>
 <contactref element="R2" pad="P$1"/>
+<contactref element="C5" pad="2"/>
+<contactref element="PS7" pad="1"/>
+<wire x1="68.712" y1="42.095" x2="69" y2="41.807" width="0.3048" layer="1"/>
+<wire x1="69" y1="41.807" x2="69" y2="41" width="0.3048" layer="1"/>
+<via x="69" y="41" extent="1-16" drill="0.35"/>
 </signal>
 <signal name="2V8-">
@@
 <wire x1="65" y1="48.5" x2="65" y2="49.5" width="0.3048" layer="1"/>
 </signal>
+<signal name="N$40">
+<contactref element="C48" pad="2"/>
+<contactref element="C5" pad="1"/>
+<wire x1="69" y1="48.55" x2="69" y2="49.85" width="0.3048" layer="1"/>
+</signal>
 </signals>

Commit message: use 4x22uF 0805 caps instead of 100uF tants
Parts:
- removed C45, C56: 100uF, SparkFun-Passives:VISHAY_C
- added C58, C6, C61, C62, C63, C64, C65, C66, C67, C68, C69, C70, C71, C72, C77, C78, C79, C80, C81, C82, C83, C84: 22uF, Nordic_nRF:RESC0805_N
- C15, C24, C33, C42, C51: value 100uF -> 22uF; device SparkFun-Passives:VISHAY_C -> Nordic_nRF:RESC0805_N
- C5: value 0.1uF -> 22uF; device Nordic_nRF:RESC0402_N -> Nordic_nRF:RESC0805_N
- moved C15 59.2 mm to (25.0, 15.0), turned to 180 degrees
- moved C2 57.6 mm to (6.00, 7.00), turned to 0 degrees
- moved C24 41.3 mm to (25.0, 18.0), turned to 180 degrees
- moved C5 28.5 mm to (61.0, 23.0), turned to 270 degrees
- moved C33 28.0 mm to (25.0, 12.0), turned to 180 degrees
- moved C42 17.0 mm to (25.0, 9.00), turned to 180 degrees
- moved J1 4.12 mm to (2.00, 5.00), turned to 180 degrees
- moved C51 1.41 mm to (67.0, 23.0), turned to 270 degrees
Connections:
- removed net N$2: C1.2, C2.1
- removed net N$40: C48.2, C5.1
- net 1V5: now also C65.1, C66.1, C67.1, C68.1; no longer C15.+
- net 2V4: now also C77.1, C78.1, C79.1, C80.1; no longer C24.+
- net 2V8+: now also C61.1, C62.1, C63.1, C64.1; no longer C42.+
- net 2V8-: now also C15.2, C24.2, C33.2, C42.2; no longer C56.-
- net 2V8D: now also C69.1, C70.1, C71.1, C72.1; no longer C33.+
- net 3V7: now also C81.1, C82.1, C83.1, C84.1; no longer C45.+
- net 5V: now also C2.1, C5.1, C51.1, C58.1, C6.1; no longer C51.+
- net GND: now also C1.2, C15.1, C24.1, C33.1, C42.1, C48.2, C51.2, C58.2, C6.2, C61.2, C62.2, C63.2, C64.2, C65.2, C66.2, C67.2, C68.2, C69.2, C70.2, C71.2, C72.2, C77.2, C78.2, C79.2, C80.2, C81.2, C82.2, C83.2, C84.2; no longer C15.-, C24.-, C33.-, C42.-, C45.-, C51.-, C56.+
Routing:
- net GND: track 143.8 -> 196.4 mm, vias 48 -> 42
- net 3V7: track 48.9 -> 63.6 mm
- net 2V8+: track 48.6 -> 62.1 mm
- net 1V5: track 47.9 -> 61.0 mm
- net 2V8D: track 48.8 -> 61.9 mm
- net 2V4: track 60.0 -> 72.7 mm
- net 5V: track 260.3 -> 271.4 mm
- net 2V8-: track 92.7 -> 103.5 mm, vias 8 -> 7
- net N$2: track 2.40 -> 0.00 mm
- net N$40: track 1.30 -> 0.00 mm
Other:
- board text removed: "+"
- board text removed: "-"

Commit message: add another 12V cap
Parts:
- added C45: 0.1uF, Nordic_nRF:RESC0402_N
Connections:
- new net N$2: C45.1, C48.2
- net GND: now also C45.2; no longer C48.2
Routing:
- net N$2: track 0.00 -> 1.30 mm
Changed lines of the file:
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@@
 <element name="C83" library="Nordic_nRF" library_urn="urn:adsk.eagle:library:169009" package="RESC0805_N" package3d_urn="urn:adsk.eagle:package:2593736/1" value="22uF" x="30" y="89" smashed="yes" rot="R180"/>
 <element name="C84" library="Nordic_nRF" library_urn="urn:adsk.eagle:library:169009" package="RESC0805_N" package3d_urn="urn:adsk.eagle:package:2593736/1" value="22uF" x="30" y="86" smashed="yes" rot="R180"/>
+<element name="C45" library="Nordic_nRF" library_urn="urn:adsk.eagle:library:169009" package="RESC0402_N" package3d_urn="urn:adsk.eagle:package:2593732/1" value="0.1uF" x="69" y="50.4" smashed="yes" rot="R90">
+<attribute name="LCSC" value="C307331" x="69" y="50.4" size="0.8128" layer="27" rot="R90" display="off"/>
+</element>
 </elements>
 <signals>
@@
 <contactref element="C1" pad="2"/>
 <contactref element="C2" pad="2"/>
-<contactref element="C48" pad="2"/>
 <contactref element="C15" pad="1"/>
 <contactref element="C24" pad="1"/>
@@
 <wire x1="70" y1="22" x2="70" y2="17.73" width="1.27" layer="1"/>
 <wire x1="70" y1="17.73" x2="69.27" y2="17" width="1.27" layer="1"/>
+<contactref element="C45" pad="2"/>
 </signal>
 <signal name="2V8-">
@@
 <wire x1="65" y1="48.5" x2="65" y2="49.5" width="0.3048" layer="1"/>
 </signal>
+<signal name="N$2">
+<contactref element="C48" pad="2"/>
+<contactref element="C45" pad="1"/>
+<wire x1="69" y1="48.55" x2="69" y2="49.85" width="0.3048" layer="1"/>
+</signal>
 </signals>
