File: power board/haasoscope_pro_power_board - 5V.brd (EAGLE design)
At the start: 77.5 x 97.5 mm, 147 parts, among them CN1 12Vin, IC11 TPS7A7200RGTR, IC12 TPS7A7200RGTR, IC14 TPS7A7200RGTR, IC3 TPS7A7200RGTR, IC5 TPS72325DBVR, IC7 TPS7A7200RGTR, IC9 TPS7A7200RGTR, J1 2p-2.54, J10 2p-2.54, J11 2p-2.54, J12 2p-2.54, J13 2p-2.54, J14 2p-2.54, J15 2p-2.54, J16 8pin, J17 2p-2.54, J18 2p-2.54, J19 2p-2.54, J2 2p-2.54, J20 2p-2.54, J3 2p-2.54, J4 2p-2.54, J5 2p-2.54, J6 2p-2.54, J7 2p-2.54, J8 2p-2.54, J9 2p-2.54

Commit message: add another 12V 10uF cap
Parts:
- added C56, C59, C60, C73: 10uF, Nordic_nRF:RESC0805_N
Connections:
- new net N$15: C56.2, C60.1
- new net N$40: C59.2, C73.1
- net 12V: now also C56.1, C59.1
- net GND: now also C60.2, C73.2
Routing:
- net 12V: track 60.7 -> 68.3 mm
- net N$15: track 0.00 -> 3.04 mm
- net N$40: track 0.00 -> 3.04 mm
Changed lines of the file:
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@@
 <attribute name="LCSC" value="C307331" x="69" y="50.4" size="0.8128" layer="27" rot="R90" display="off"/>
 </element>
+<element name="C56" library="Nordic_nRF" library_urn="urn:adsk.eagle:library:169009" package="RESC0805_N" package3d_urn="urn:adsk.eagle:package:2593736/1" value="10uF" x="65" y="65" smashed="yes" rot="R180"/>
+<element name="C59" library="Nordic_nRF" library_urn="urn:adsk.eagle:library:169009" package="RESC0805_N" package3d_urn="urn:adsk.eagle:package:2593736/1" value="10uF" x="65" y="62" smashed="yes" rot="R180"/>
+<element name="C60" library="Nordic_nRF" library_urn="urn:adsk.eagle:library:169009" package="RESC0805_N" package3d_urn="urn:adsk.eagle:package:2593736/1" value="10uF" x="65" y="68" smashed="yes"/>
+<element name="C73" library="Nordic_nRF" library_urn="urn:adsk.eagle:library:169009" package="RESC0805_N" package3d_urn="urn:adsk.eagle:package:2593736/1" value="10uF" x="65" y="59" smashed="yes"/>
 </elements>
 <signals>
@@
 <wire x1="70" y1="17.73" x2="69.27" y2="17" width="1.27" layer="1"/>
 <contactref element="C45" pad="2"/>
+<contactref element="C60" pad="2"/>
+<contactref element="C73" pad="2"/>
 </signal>
 <signal name="2V8-">
@@
 <wire x1="65.1321" y1="71.65835" x2="65.1321" y2="71.8829" width="1.27" layer="1"/>
 <wire x1="65.1321" y1="71.8829" x2="64.205" y2="72.81" width="1.27" layer="1"/>
-<wire x1="70.2619" y1="46.55615" x2="70.2619" y2="66.52855" width="1.27" layer="1"/>
+<wire x1="70.2619" y1="46.55615" x2="70.2619" y2="66" width="1.27" layer="1"/>
+<wire x1="70.2619" y1="66" x2="70.2619" y2="66.52855" width="1.27" layer="1"/>
 <wire x1="70.2619" y1="66.52855" x2="65.1321" y2="71.65835" width="1.27" layer="1"/>
 <wire x1="64.205" y1="72.81" x2="63.4" y2="73.615" width="1.27" layer="1"/>
@@
 <wire x1="62.3" y1="88" x2="62.4126" y2="88.1126" width="1.27" layer="1"/>
 <wire x1="62.4126" y1="88.1126" x2="66.40115" y2="88.1126" width="1.27" layer="1"/>
+<contactref element="C56" pad="1"/>
+<contactref element="C59" pad="1"/>
+<wire x1="66.1" y1="65" x2="66.1" y2="62" width="1.27" layer="1"/>
+<wire x1="66.1" y1="65" x2="67.1" y2="66" width="1.27" layer="1"/>
+<wire x1="67.1" y1="66" x2="70.2619" y2="66" width="1.27" layer="1"/>
 </signal>
 <signal name="N$32">
@@
 <wire x1="69" y1="48.55" x2="69" y2="49.85" width="0.3048" layer="1"/>
 </signal>
+<signal name="N$15">
+<contactref element="C56" pad="2"/>
+<contactref element="C60" pad="1"/>
+<wire x1="64" y1="65" x2="64" y2="67.9" width="1.27" layer="1"/>
+<wire x1="64" y1="67.9" x2="63.9" y2="68" width="1.27" layer="1"/>
+</signal>
+<signal name="N$40">
+<contactref element="C59" pad="2"/>
+<contactref element="C73" pad="1"/>
+<wire x1="63.9" y1="59" x2="64" y2="59.1" width="1.27" layer="1"/>
+<wire x1="64" y1="59.1" x2="64" y2="62" width="1.27" layer="1"/>
+</signal>
 </signals>

Commit message: 2.4->2.2V for 1.9V reg, to reduce heat add vias in regulator gnd pads, to dissipate heat
Parts:
- removed J17, J18, J19: 2p-2.54, Seeed-Connector:H2-2.54
- R6: value 100k -> 82k
- moved J3 4.02 mm to (69.3, 71.5)
- moved C52 4.02 mm to (65.7, 15.6)
- moved C19 4.02 mm to (16.5, 59.7)
- moved C20 4.02 mm to (14.0, 59.7)
- moved IC7 4.02 mm to (22.9, 59.7)
- moved C13 4.02 mm to (10.2, 17.3)
- moved C15 4.02 mm to (28.8, 13.7)
- moved C2 4.02 mm to (9.80, 5.70)
- moved C24 4.02 mm to (28.8, 16.7)
- moved C3 4.02 mm to (66.1, 89.3)
- moved C33 4.02 mm to (28.8, 10.7)
- moved C35 4.02 mm to (8.89, 26.7)
- moved C42 4.02 mm to (28.8, 7.70)
- moved C47 4.02 mm to (23.8, 27.7)
- moved C57 4.02 mm to (23.8, 13.7)
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Connections:
- net 2V4 renamed 2V2
- removed net N$10: IC7.5, J17.2
- removed net N$8: IC3.5, J19.2
- removed net N$9: IC9.5, J18.2
- net GND: no longer J17.1, J18.1, J19.1
Routing:
- net N$8: track 4.93 -> 0.00 mm
- net N$9: track 4.69 -> 0.00 mm
- net N$10: track 4.45 -> 0.00 mm
- net GND: vias 42 -> 48
Other:
- board text added: "2.2V out GND"
- board text added: "Haasoscope Pro Power board, v1.21 by Dr. Andy Haas"
- board text removed: "+0.1V"
- board text removed: "2.4V out GND"
- board text removed: "Haasoscope Pro Power board, v1.2 by Dr. Andy Haas"
