File: input board/haasoscope_pro_input_board.sch (EAGLE design)
At the start: 51 parts, among them IC1 LMH5401IRMST, IC2 LMH6401IRMZR, IC3 SN74AVC4T774PWR, IC4 OPA693ID, IC6 DAC8562SDGSR, IC7 TLV9102IPWR, J1 8pin, J3 2X4P-2.54, J4 8pin

Commit message: power connector etc
Parts:
- removed J3: 2X4P-2.54, Seeed-Connector:DIP-BLACK-FEMALE-HEADER(2X4P-2.54)
Connections:
- net 2V5OUT renamed 2V5DACOUT
- net 3V3: no longer J4.7
- net AMPSCLK: no longer J3.8
- net AMPSCS: no longer J3.7
- net AMPSDI: no longer J3.6
- net AMPSDO: no longer J3.5
- net GND: no longer J3.1, J3.4, J4.8
- net VS+: now also J4.7; no longer J3.2
- net VS-: now also J4.8; no longer J3.3
Changed lines of the file:
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@@
 <part name="AOUT-" library="con-coax" library_urn="urn:adsk.eagle:library:133" deviceset="BU-SMB-V" device="" package3d_urn="urn:adsk.eagle:package:6209/1"/>
 <part name="SUPPLY41" library="supply2" library_urn="urn:adsk.eagle:library:372" deviceset="GND" device=""/>
-<part name="J3" library="Seeed-Connector" library_urn="urn:adsk.eagle:library:478" deviceset="DIP-BLACK-FEMALE-HEADER(2X4P-2.54)" device="" package3d_urn="urn:adsk.eagle:package:33148/1" value="2X4P-2.54"/>
 <part name="C1" library="MF_Passives" deviceset="CAPACITOR_NP" device="_0402" value="0.1uF"/>
 <part name="C2" library="MF_Passives" deviceset="CAPACITOR_NP" device="_0402" value="0.1uF"/>
@@
 </instance>
 <instance part="SUPPLY41" gate="GND" x="203.2" y="83.82" smashed="yes"/>
-<instance part="J3" gate="G$1" x="143.764" y="19.05" smashed="yes"/>
 <instance part="C1" gate="G$1" x="132.08" y="106.68" smashed="yes">
 <attribute name="NAME" x="134.62" y="108.204" size="1.016" layer="95" font="vector" align="top-left"/>
@@
 <attribute name="VALUE" x="252.73" y="35.56" size="1.778" layer="96" align="center-left"/>
 </instance>
-<instance part="J4" gate="G$1" x="322.58" y="22.86" smashed="yes" rot="R180"/>
+<instance part="J4" gate="G$1" x="25.4" y="27.94" smashed="yes" rot="R180"/>
 <instance part="SUPPLY15" gate="GND" x="347.98" y="15.24" smashed="yes"/>
 <instance part="SUPPLY16" gate="GND" x="337.82" y="15.24" smashed="yes"/>
@@
 </segment>
 <segment>
-<label x="129.54" y="22.86" size="1.778" layer="95"/>
-<pinref part="J3" gate="G$1" pin="1"/>
-<wire x1="134.874" y1="22.86" x2="129.54" y2="22.86" width="0.1524" layer="91"/>
-</segment>
-<segment>
-<label x="129.54" y="15.24" size="1.778" layer="95"/>
-<pinref part="J3" gate="G$1" pin="4"/>
-<wire x1="134.874" y1="15.24" x2="129.54" y2="15.24" width="0.1524" layer="91"/>
-</segment>
-<segment>
 <pinref part="IC1" gate="G$1" pin="PD"/>
 <wire x1="162.56" y1="86.36" x2="172.72" y2="86.36" width="0.1524" layer="91"/>
@@
 <segment>
 <pinref part="J4" gate="G$1" pin="2"/>
-<wire x1="317.5" y1="27.94" x2="307.34" y2="27.94" width="0.1524" layer="91"/>
-<label x="307.34" y="27.94" size="1.778" layer="95"/>
+<wire x1="20.32" y1="33.02" x2="10.16" y2="33.02" width="0.1524" layer="91"/>
+<label x="10.16" y="33.02" size="1.778" layer="95"/>
 </segment>
 <segment>
@@
 </segment>
 <segment>
-<pinref part="J4" gate="G$1" pin="8"/>
-<wire x1="317.5" y1="12.7" x2="307.34" y2="12.7" width="0.1524" layer="91"/>
-<label x="307.34" y="12.7" size="1.778" layer="95"/>
-</segment>
-<segment>
 <pinref part="SUPPLY16" gate="GND" pin="GND"/>
 <pinref part="C9" gate="G$1" pin="P$2"/>
@@
 <net name="VS+" class="0">
 <segment>
-<label x="129.54" y="20.32" size="1.778" layer="95"/>
-<pinref part="J3" gate="G$1" pin="2"/>
-<wire x1="134.874" y1="20.32" x2="129.54" y2="20.32" width="0.1524" layer="91"/>
-</segment>
-<segment>
 <pinref part="C1" gate="G$1" pin="P$1"/>
 <wire x1="132.08" y1="109.22" x2="132.08" y2="114.3" width="0.1524" layer="91"/>
@@
 <label x="208.28" y="-27.94" size="1.778" layer="95"/>
 </segment>
+<segment>
+<pinref part="J4" gate="G$1" pin="7"/>
+<wire x1="20.32" y1="20.32" x2="10.16" y2="20.32" width="0.1524" layer="91"/>
+<label x="10.16" y="20.32" size="1.778" layer="95"/>
+</segment>
 </net>
 <net name="VS-" class="0">
-<segment>
-<label x="129.54" y="17.78" size="1.778" layer="95"/>
-<pinref part="J3" gate="G$1" pin="3"/>
-<wire x1="134.874" y1="17.78" x2="129.54" y2="17.78" width="0.1524" layer="91"/>
-</segment>
 <segment>
 <pinref part="C2" gate="G$1" pin="P$1"/>
@@
 <wire x1="218.44" y1="-33.02" x2="218.44" y2="-27.94" width="0.1524" layer="91"/>
 <label x="218.44" y="-27.94" size="1.778" layer="95"/>
+</segment>
+<segment>
+<pinref part="J4" gate="G$1" pin="8"/>
+<wire x1="20.32" y1="17.78" x2="10.16" y2="17.78" width="0.1524" layer="91"/>
+<label x="10.16" y="17.78" size="1.778" layer="95"/>
 </segment>
 </net>
@@
 </segment>
 <segment>
-<wire x1="165.1" y1="17.78" x2="152.654" y2="17.78" width="0.1524" layer="91"/>
-<label x="154.94" y="17.78" size="1.778" layer="95"/>
-<pinref part="J3" gate="G$1" pin="6"/>
-</segment>
-<segment>
 <pinref part="IC3" gate="G$1" pin="B3"/>
 <wire x1="274.32" y1="20.32" x2="284.48" y2="20.32" width="0.1524" layer="91"/>
@@
 </segment>
 <segment>
-<wire x1="165.1" y1="15.24" x2="152.654" y2="15.24" width="0.1524" layer="91"/>
-<label x="154.94" y="15.24" size="1.778" layer="95"/>
-<pinref part="J3" gate="G$1" pin="5"/>
-</segment>
-<segment>
 <pinref part="IC3" gate="G$1" pin="B4"/>
 <wire x1="274.32" y1="17.78" x2="284.48" y2="17.78" width="0.1524" layer="91"/>
@@
 </segment>
 <segment>
-<wire x1="165.1" y1="22.86" x2="152.654" y2="22.86" width="0.1524" layer="91"/>
-<label x="154.94" y="22.86" size="1.778" layer="95"/>
-<pinref part="J3" gate="G$1" pin="8"/>
-</segment>
-<segment>
 <pinref part="IC3" gate="G$1" pin="B1"/>
 <wire x1="274.32" y1="25.4" x2="284.48" y2="25.4" width="0.1524" layer="91"/>
@@
 <pinref part="IC2" gate="G$1" pin="!CS"/>
 <label x="312.42" y="73.66" size="1.778" layer="95"/>
-</segment>
-<segment>
-<wire x1="165.1" y1="20.32" x2="152.654" y2="20.32" width="0.1524" layer="91"/>
-<label x="154.94" y="20.32" size="1.778" layer="95"/>
-<pinref part="J3" gate="G$1" pin="7"/>
 </segment>
 <segment>
@@
 <segment>
 <pinref part="J4" gate="G$1" pin="3"/>
-<wire x1="307.34" y1="25.4" x2="317.5" y2="25.4" width="0.1524" layer="91"/>
-<label x="307.34" y="25.4" size="1.778" layer="95"/>
+<wire x1="10.16" y1="30.48" x2="20.32" y2="30.48" width="0.1524" layer="91"/>
+<label x="10.16" y="30.48" size="1.778" layer="95"/>
 </segment>
 </net>
@@
 <segment>
 <pinref part="J4" gate="G$1" pin="4"/>
-<wire x1="307.34" y1="22.86" x2="317.5" y2="22.86" width="0.1524" layer="91"/>
-<label x="307.34" y="22.86" size="1.778" layer="95"/>
+<wire x1="10.16" y1="27.94" x2="20.32" y2="27.94" width="0.1524" layer="91"/>
+<label x="10.16" y="27.94" size="1.778" layer="95"/>
 </segment>
 </net>
@@
 <segment>
 <pinref part="J4" gate="G$1" pin="5"/>
-<wire x1="317.5" y1="20.32" x2="307.34" y2="20.32" width="0.1524" layer="91"/>
-<label x="307.34" y="20.32" size="1.778" layer="95"/>
+<wire x1="20.32" y1="25.4" x2="10.16" y2="25.4" width="0.1524" layer="91"/>
+<label x="10.16" y="25.4" size="1.778" layer="95"/>
 </segment>
 </net>
@@
 <segment>
 <pinref part="J4" gate="G$1" pin="6"/>
-<wire x1="317.5" y1="17.78" x2="307.34" y2="17.78" width="0.1524" layer="91"/>
-<label x="307.34" y="17.78" size="1.778" layer="95"/>
+<wire x1="20.32" y1="22.86" x2="10.16" y2="22.86" width="0.1524" layer="91"/>
+<label x="10.16" y="22.86" size="1.778" layer="95"/>
 </segment>
 </net>
@@
 <segment>
 <pinref part="J4" gate="G$1" pin="1"/>
-<pinref part="IC3" gate="G$1" pin="VCCA"/>
-<wire x1="274.32" y1="30.48" x2="317.5" y2="30.48" width="0.1524" layer="91"/>
-<label x="307.34" y="30.48" size="1.778" layer="95"/>
+<wire x1="10.16" y1="35.56" x2="20.32" y2="35.56" width="0.1524" layer="91"/>
+<label x="10.16" y="35.56" size="1.778" layer="95"/>
 </segment>
 <segment>
@@
 <wire x1="246.38" y1="30.48" x2="236.22" y2="30.48" width="0.1524" layer="91"/>
 <label x="236.22" y="30.48" size="1.778" layer="95"/>
-</segment>
-<segment>
-<pinref part="J4" gate="G$1" pin="7"/>
-<wire x1="317.5" y1="15.24" x2="307.34" y2="15.24" width="0.1524" layer="91"/>
-<label x="307.34" y="15.24" size="1.778" layer="95"/>
 </segment>
 <segment>
@@
 <wire x1="20.32" y1="-10.16" x2="10.16" y2="-10.16" width="0.1524" layer="91"/>
 <label x="10.16" y="-10.16" size="1.778" layer="95"/>
+</segment>
+<segment>
+<pinref part="IC3" gate="G$1" pin="VCCA"/>
+<wire x1="274.32" y1="30.48" x2="284.48" y2="30.48" width="0.1524" layer="91"/>
+<label x="279.4" y="30.48" size="1.778" layer="95"/>
 </segment>
 </net>
@@
 </segment>
 </net>
-<net name="2V5OUT" class="0">
+<net name="2V5DACOUT" class="0">
 <segment>
 <pinref part="IC6" gate="G$1" pin="VREFIN/VREFOUT"/>

Commit message: power connector etc
Parts:
- added R21, R22: 0, MF_Passives:RESISTOR_0402
- AMPOUT+, AMPOUT-: value BU-SMB-V -> (none); device con-coax:BU-SMB-V -> adafruit:SMACONNECTOR_EDGE
Connections:
- new net N$4: AOUT-.1, R22.P$2
- new net N$6: AOUT+.1, R21.P$2
- net AMPOUTSMA_N: now also AMPOUT-.ANT; no longer AMPOUT-.1
- net AMPOUTSMA_P: now also AMPOUT+.ANT; no longer AMPOUT+.1
- net AOUTSMA_N: now also R22.P$1; no longer AOUT-.1
- net AOUTSMA_P: now also R21.P$1; no longer AOUT+.1
- net GND: now also AMPOUT+.GND1, AMPOUT+.GND2, AMPOUT+.GND3, AMPOUT+.GND4, AMPOUT-.GND1, AMPOUT-.GND2, AMPOUT-.GND3, AMPOUT-.GND4; no longer AMPOUT+.2, AMPOUT-.2
Other:
- moved on the sheet: AOUT+, AOUT-

Commit message: minor-fix ampout for jlcpcb
Parts:
- AMPOUT+: value (none) -> out+
- AMPOUT-: value (none) -> out-
Changed lines of the file:
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@@
 <part name="R20" library="MF_Passives" deviceset="RESISTOR" device="_0402" value="1k"/>
 <part name="J1" library="SparkFun-Connectors" library_urn="urn:adsk.eagle:library:513" deviceset="CONN_08" device="&quot;" package3d_urn="urn:adsk.eagle:package:38138/1" value="8pin"/>
-<part name="AMPOUT-" library="adafruit" deviceset="SMACONNECTOR" device="_EDGE"/>
-<part name="AMPOUT+" library="adafruit" deviceset="SMACONNECTOR" device="_EDGE"/>
+<part name="AMPOUT-" library="adafruit" deviceset="SMACONNECTOR" device="_EDGE" value="out-"/>
+<part name="AMPOUT+" library="adafruit" deviceset="SMACONNECTOR" device="_EDGE" value="out+"/>
 <part name="SUPPLY7" library="supply2" library_urn="urn:adsk.eagle:library:372" deviceset="GND" device=""/>
 <part name="SUPPLY8" library="supply2" library_urn="urn:adsk.eagle:library:372" deviceset="GND" device=""/>

Commit message: working dac offset
Parts:
- removed R14: 0, MF_Passives:RESISTOR_0402
Connections:
- net AOFFSET: no longer R14.P$2
- net GND: no longer R14.P$1
Changed lines of the file:
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@@
 <part name="R13" library="MF_Passives" deviceset="RESISTOR" device="_0402" value="1k"/>
 <part name="SUPPLY18" library="supply2" library_urn="urn:adsk.eagle:library:372" deviceset="GND" device=""/>
-<part name="R14" library="MF_Passives" deviceset="RESISTOR" device="_0402" value="0"/>
-<part name="SUPPLY2" library="supply2" library_urn="urn:adsk.eagle:library:372" deviceset="GND" device=""/>
 <part name="R15" library="MF_Passives" deviceset="RESISTOR" device="_0402" value="0"/>
 <part name="IC4" library="OPA693ID" deviceset="OPA693ID" device=""/>
@@
 </instance>
 <instance part="SUPPLY18" gate="GND" x="193.04" y="12.7" smashed="yes"/>
-<instance part="R14" gate="G$1" x="96.52" y="71.12" smashed="yes" rot="R180">
-<attribute name="NAME" x="97.536" y="68.58" size="1.016" layer="95" font="vector" rot="R90" align="top-left"/>
-<attribute name="VALUE" x="97.536" y="73.66" size="1.016" layer="96" font="vector" rot="R270"/>
-</instance>
-<instance part="SUPPLY2" gate="GND" x="96.52" y="63.5" smashed="yes"/>
 <instance part="R15" gate="G$1" x="93.98" y="71.12" smashed="yes" rot="R180">
 <attribute name="NAME" x="94.996" y="68.58" size="1.016" layer="95" font="vector" rot="R90" align="top-left"/>
@@
 <pinref part="R13" gate="G$1" pin="P$1"/>
 <pinref part="SUPPLY18" gate="GND" pin="GND"/>
-</segment>
-<segment>
-<pinref part="R14" gate="G$1" pin="P$1"/>
-<pinref part="SUPPLY2" gate="GND" pin="GND"/>
 </segment>
 <segment>
@@
 <segment>
 <pinref part="R5" gate="G$1" pin="P$1"/>
-<wire x1="101.6" y1="76.2" x2="96.52" y2="76.2" width="0.1524" layer="91"/>
+<wire x1="101.6" y1="76.2" x2="93.98" y2="76.2" width="0.1524" layer="91"/>
 <label x="91.44" y="76.2" size="1.778" layer="95"/>
-<pinref part="R14" gate="G$1" pin="P$2"/>
-<wire x1="96.52" y1="76.2" x2="93.98" y2="76.2" width="0.1524" layer="91"/>
-<junction x="96.52" y="76.2"/>
 <pinref part="R15" gate="G$1" pin="P$2"/>
 <wire x1="93.98" y1="76.2" x2="91.44" y2="76.2" width="0.1524" layer="91"/>
