File: clock board/haasoscope_pro_clock_board.brd (EAGLE design)
At the start: 127 x 74 mm, 8 parts, among them IC1 LMX2582RHAT, J3 2X4P-2.54

Commit message: initial adf4350
Parts:
- removed IC1: LMX2582RHAT, LMX2582RHAT:QFN50P600X600X100-41N
- added C28, C29, C37, C57, C58: 1U, capacitor:CAPC1608X90N
- added C30: 10N, capacitor:CAPC1005X55N
- added C31: 22U, capacitor:CAPMP7343X430N
- added C38, C40, C42, C45, C46, C48, C50, C52: 10P, capacitor:CAPC1005X55N
- added C39, C41, C43, C44, C47, C49, C51, C53, C56: 100N, capacitor:CAPC1005X55N
- added C54, C55: 120P, capacitor:CAPC1005X55N
- added C59, C60: 100P, capacitor:CAPC1005X55N
- added C61: 3N3, capacitor:CAPC1608X90N
- added C62: 47N, capacitor:CAPC1608X90N
- added C63: 1N5, capacitor:CAPC1608X90N
- added FB2: FB0603, inductor:INDC1608X95N
- added R10, R11, R13, R9: 10K, resistor:RESC1608X55N
- added R14: 316, resistor:RESC1608X55N
- added R18: 681, resistor:RESC1608X55N
- added R22, R7: 0, resistor:RESC1608X55N
- added R23: DNI, resistor:RESC1608X55N
- added R24, R25: 49R9, resistor:RESC1005X40N
- added R8: 5K11, resistor:RESC1608X55N
- added U4: ADF4350BCPZ, analog_devices:QFN50P500X500X100-33V2N
- added U5, U6: ADP150AUJZ-3.3, analog_devices:SOT95P280X110-5N
- added Y2: XO_E5X3, oscillator:OSCSC254P320X500X120-4N
Connections:
- new net 3V3: C29.2, C38.2, C39.2, C40.1, C41.1, C42.2, C43.2, C44.2, C45.2, C46.2, C47.2, FB2.2, R9.2, U4.10, U4.16, U4.17, U4.26, U4.28, U4.32, U4.6, U5.5
- new net ADFCE: R9.1, U4.4
- new net ADFCLK: R10.2, U4.1
- new net ADFDATA: R11.2, U4.2
- new net ADFLE: R13.2, U4.3
- new net LD: U4.25
- new net MUXOUT: U4.30
- new net N$13: R7.1, Y2.3
- new net N$18: C48.2, C49.2, U4.19
- new net N$19: C50.2, C51.2, U4.23
- new net N$31: R8.1, U4.22
- new net N$4: C30.2, C37.2, FB2.1, Y2.1, Y2.4
- new net N$40: C60.2
- new net N$41: C59.2
- new net N$42: C61.2, C62.1, R18.2, U4.7
- new net N$44: C62.2, R14.1
- new net N$45: R14.2, R22.2, R23.1
- new net N$46: R23.2, U4.5
- new net REFOUTA_N: C60.1, R25.1, U4.13
- new net REFOUTA_P: C59.1, R24.1, U4.12
- new net REF_CLK: R7.2, U4.29
- new net VIN: C28.2, C31.1, C57.2, U5.1, U5.3, U6.1, U6.3
- new net VOUT: C54.2, C55.2, C56.2, C58.2, R24.2, R25.2, U6.5
- new net VREF: C52.1, C53.1, U4.24
- new net VTUNE: C63.2, R18.1, U4.20
- net GND: now also C28.1, C29.1, C30.1, C31.2, C37.1, C38.1, C39.1, C40.2, C41.2, C42.1, C43.1, C44.1, C45.1, C46.1, C47.1, C48.1, C49.1, C50.1, C51.1, C52.2, C53.2, C54.1, C55.1, C56.1, C57.1, C58.1, C61.1, C63.1, R10.1, R11.1, R13.1, R22.1, R8.2, U4.11, U4.18, U4.21, U4.27, U4.31, U4.8, U4.9, U4.PAD@1_1, U4.PAD@1_2, U4.PAD@1_3, U4.PAD@2_1, U4.PAD@2_2, U4.PAD@2_3, U4.PAD@3_1, U4.PAD@3_2, U4.PAD@3_3, U5.2, U6.2, Y2.2
Routing:
- added copper zone on layer 15, net 3V3
- added copper zone on layer 1, net GND

Commit message: v1.0
Parts:
- removed AOUT+, AOUT-: BU-SMB-V, con-coax:BU-SMB-V
- removed C28, C29, C37, C57, C58: 1U, capacitor:CAPC1608X90N
- removed C30: 10N, capacitor:CAPC1005X55N
- removed C31: 22U, capacitor:CAPMP7343X430N
- removed C38, C40, C42, C45, C46, C48, C50, C52: 10P, capacitor:CAPC1005X55N
- removed C39, C41, C43, C44, C47, C49, C51, C53, C56: 100N, capacitor:CAPC1005X55N
- removed C54, C55: 120P, capacitor:CAPC1005X55N
- removed C59, C60: 100P, capacitor:CAPC1005X55N
- removed C61: 3N3, capacitor:CAPC1608X90N
- removed C62: 47N, capacitor:CAPC1608X90N
- removed C63: 1N5, capacitor:CAPC1608X90N
- removed FB2: FB0603, inductor:INDC1608X95N
- removed J3: 2X4P-2.54, Seeed-Connector:H2X4-2.54
- removed R13: 10K, resistor:RESC1608X55N
- removed R14: 316, resistor:RESC1608X55N
- removed R18: 681, resistor:RESC1608X55N
- removed R22: 0, resistor:RESC1608X55N
- removed R23: DNI, resistor:RESC1608X55N
- removed R24, R25: 49R9, resistor:RESC1005X40N
- removed U5, U6: ADP150AUJZ-3.3, analog_devices:SOT95P280X110-5N
- removed Y2: XO_E5X3, oscillator:OSCSC254P320X500X120-4N
- added C10, C11: 0.1nF, MF_Passives:C0402
- added C12, C13: 1nF, MF_Passives:C0402
- added C14: 2.7nF, MF_Passives:C0402
- added C15: 47nF, MF_Passives:C0402
- added C16: 680pF, MF_Passives:C0402
- added C3, C4, C5, C6, C7, C8, C9: 0.1uF, MF_Passives:C0402
- added J4: 8pin, SparkFun-Connectors:1X08
- added R1: 47, MF_Passives:R0402
- added R4, R5, R6: 10k, MF_Passives:R0402
- added REFRFIN, RFAOUT+, RFAOUT-: (no value), adafruit:SMA_EDGELAUNCH
- R10: value 10K -> 1k; device resistor:RESC1608X55N -> MF_Passives:R0402
- R11: value 10K -> 360; device resistor:RESC1608X55N -> MF_Passives:R0402
- R2: value 40 -> 0
- R3: value 40 -> 47
- R7: value 0 -> 10k; device resistor:RESC1608X55N -> MF_Passives:R0402
- R8: value 5K11 -> 5.1k; device resistor:RESC1608X55N -> MF_Passives:R0402
- R9: value 10K -> 47; device resistor:RESC1608X55N -> MF_Passives:R0402
- moved R9 94.8 mm to (12.0, 45.0), turned to 90 degrees
- moved R11 74.5 mm to (33.0, 61.0)
- moved R8 73.5 mm to (32.0, 52.0), turned to 0 degrees
- moved U4 72.2 mm to (34.0, 46.0)
- moved R10 71.5 mm to (33.0, 58.0)
- moved R7 56.8 mm to (41.0, 26.0), turned to 180 degrees
- moved C2 26.2 mm to (28.0, 47.0)
- moved R2 25.6 mm to (43.0, 53.0), turned to 270 degrees
- moved R3 23.2 mm to (42.0, 45.0), turned to 90 degrees
- moved C1 15.7 mm to (39.0, 49.0), turned to 90 degrees
Connections:
- removed net 3V3: C29.2, C38.2, C39.2, C40.1, C41.1, C42.2, C43.2, C44.2, C45.2, C46.2, C47.2, FB2.2, R9.2, U4.10, U4.16, U4.17, U4.26, U4.28, U4.32, U4.6, U5.5
- removed net N$13: R7.1, Y2.3
- removed net N$4: C30.2, C37.2, FB2.1, Y2.1, Y2.4
- removed net N$40: C60.2
- removed net N$41: C59.2
- removed net N$42: C61.2, C62.1, R18.2, U4.7
- removed net N$44: C62.2, R14.1
- removed net N$45: R14.2, R22.2, R23.1
- removed net N$46: R23.2, U4.5
- removed net REFOUTA_N: C60.1, R25.1, U4.13
- removed net REFOUTA_P: C59.1, R24.1, U4.12
- removed net VIN: C28.2, C31.1, C57.2, U5.1, U5.3, U6.1, U6.3
- removed net VS+: C1.P$1, J3.2
- removed net VS-: C2.P$1, J3.3
- new net +3V3: C1.P$1, C2.P$2, C6.P$2, C7.P$2, C8.P$1, J4.8, R2.P$1, R7.P$2, U4.10, U4.16, U4.17, U4.26, U4.28, U4.32, U4.6
- new net CPOUT: C14.P$1, R10.P$2, R11.P$1, U4.7
- new net N$3: C15.P$1, R11.P$2
- new net RFOUTASMA_N: C10.P$1, RFAOUT-.P
- new net RFOUTASMA_P: C11.P$1, RFAOUT+.P
- new net RFOUTA_N: C10.P$2, R1.P$1, U4.13
- new net RFOUTA_P: C11.P$2, R3.P$1, U4.12
- net ADFCE: now also J4.2, R7.P$1; no longer R9.1
- net ADFCLK: now also J4.5, R6.P$2; no longer R10.2
- net ADFDATA: now also J4.4, R5.P$2; no longer R11.2
- net ADFLE: now also J4.3, R4.P$2; no longer R13.2
- net GND: now also C14.P$2, C15.P$2, C16.P$2, C2.P$1, C3.P$2, C4.P$1, C5.P$1, C6.P$1, C7.P$1, C8.P$2, C9.P$2, J4.1, R4.P$1, R5.P$1, R6.P$1, R8.P$1, R9.P$1, REFRFIN.GND@1, REFRFIN.GND@2, REFRFIN.GND@3, REFRFIN.GND@4, RFAOUT+.GND@1, RFAOUT+.GND@2, RFAOUT+.GND@3, RFAOUT+.GND@4, RFAOUT-.GND@1, RFAOUT-.GND@2, RFAOUT-.GND@3, RFAOUT-.GND@4; no longer AOUT+.2, AOUT+.3, AOUT+.4, AOUT+.5, AOUT-.2, AOUT-.3, AOUT-.4, AOUT-.5, C2.P$2, C28.1, C29.1, C30.1, C31.2, C37.1, C38.1, C39.1, C40.2, C41.2, C42.1, C43.1, C44.1, C45.1, C46.1, C47.1, C48.1, C49.1, C50.1, C51.1, C52.2, C53.2, C54.1, C55.1, C56.1, C57.1, C58.1, C61.1, C63.1, J3.1, J3.4, J3.5, J3.6, J3.7, J3.8, R10.1, R11.1, R13.1, R22.1, R8.2, U5.2, U6.2, Y2.2
- net LD: now also J4.7
- net MUXOUT: now also J4.6
- net N$1: now also C12.P$2, REFRFIN.P; no longer AOUT+.1, R2.P$2
- net N$18: now also C5.P$2; no longer C48.2, C49.2
- net N$19: now also C4.P$2; no longer C50.2, C51.2
- net N$2: now also C12.P$1, C13.P$2, R9.P$2; no longer AOUT-.1, R3.P$2
- net N$31: now also R8.P$2; no longer R8.1
- net REF_CLK: now also C13.P$1; no longer R7.2
- net VOUT: now also C9.P$1, R1.P$2, R2.P$2, R3.P$2; no longer C54.2, C55.2, C56.2, C58.2, R24.2, R25.2, U6.5
- net VREF: now also C3.P$1; no longer C52.1, C53.1
- net VTUNE: now also C16.P$1, R10.P$1; no longer C63.2, R18.1
Routing:
- net LD: track 0.00 -> 62.0 mm, vias 0 -> 2
- net MUXOUT: track 0.00 -> 57.7 mm
- net ADFCLK: track 0.00 -> 40.8 mm
- net ADFDATA: track 0.00 -> 37.6 mm
- net ADFLE: track 0.00 -> 34.7 mm
- net ADFCE: track 0.00 -> 30.5 mm
- net GND: track 0.00 -> 29.6 mm, vias 0 -> 41
- net CPOUT: track 0.00 -> 26.4 mm, vias 0 -> 2
- net +3V3: track 0.00 -> 26.2 mm, vias 0 -> 7
- net REF_CLK: track 0.00 -> 16.1 mm
- net VOUT: track 0.00 -> 11.7 mm, vias 0 -> 2
- net VTUNE: track 0.00 -> 11.5 mm
- net RFOUTASMA_P: track 0.00 -> 9.40 mm
- net RFOUTASMA_N: track 0.00 -> 9.40 mm
- net RFOUTA_N: track 0.00 -> 8.76 mm
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- added copper zone on layer 15, net +3V3
- removed copper zone on layer 15, net 3V3
Other:
- board size 127 x 74 mm -> 54 x 74 mm
- board text added: "+3V3"
- board text added: "CE"
- board text added: "CLK"
- board text added: "DATA"
- board text added: "Haasoscope Pro Clock board, v1.0 by Dr. Andy Haas August 2024"
- board text added: "LE"
- board text added: "LOCK"
- board text added: "MUXOUT"
- board text removed: "Haasoscope Pro Clock board, v1.0 by Dr. Andy Haas July 2024"
- board text removed: "VS+"
- board text removed: "VS-"

Commit message: v1.0
Parts:
- REFRFIN, RFAOUT+, RFAOUT-: value (none) -> sma
Changed lines of the file:
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@@
 </element>
 <element name="U4" library="analog_devices" package="QFN50P500X500X100-33V2N" value="ADF4350BCPZ" x="34" y="46" smashed="yes" rot="R90"/>
-<element name="RFAOUT-" library="adafruit" package="SMA_EDGELAUNCH" value="" x="53" y="54" smashed="yes" rot="R180">
+<element name="RFAOUT-" library="adafruit" package="SMA_EDGELAUNCH" value="sma" x="53" y="54" smashed="yes" rot="R180">
 <attribute name="NAME" x="46.92" y="47.015" size="1.016" layer="25" ratio="18"/>
-<attribute name="VALUE" x="47.92" y="48.92" size="0.8128" layer="27" ratio="10"/>
 </element>
-<element name="RFAOUT+" library="adafruit" package="SMA_EDGELAUNCH" value="" x="53" y="38" smashed="yes" rot="R180">
+<element name="RFAOUT+" library="adafruit" package="SMA_EDGELAUNCH" value="sma" x="53" y="38" smashed="yes" rot="R180">
 <attribute name="NAME" x="46.92" y="31.015" size="1.016" layer="25" ratio="18"/>
-<attribute name="VALUE" x="47.92" y="32.92" size="0.8128" layer="27" ratio="10"/>
 </element>
 <element name="J4" library="SparkFun-Connectors" library_urn="urn:adsk.eagle:library:513" package="1X08" package3d_urn="urn:adsk.eagle:package:38138/1" value="8pin" x="51" y="28" smashed="yes" rot="R270">
@@
 <attribute name="VOLTAGE" value="" x="45" y="44" size="1.778" layer="27" rot="R180" display="off"/>
 </element>
-<element name="REFRFIN" library="adafruit" package="SMA_EDGELAUNCH" value="" x="1" y="46" smashed="yes">
+<element name="REFRFIN" library="adafruit" package="SMA_EDGELAUNCH" value="sma" x="1" y="46" smashed="yes">
 <attribute name="NAME" x="0.92" y="52.015" size="1.016" layer="25" ratio="18"/>
-<attribute name="VALUE" x="6.08" y="51.08" size="0.8128" layer="27" ratio="10" rot="R180"/>
 </element>
 <element name="C12" library="MF_Passives" package="C0402" value="1nF" x="9" y="46" smashed="yes" rot="R180">

Commit message: add refB out, fix i/o spacing
Parts:
- removed RFAOUT+, RFAOUT-: sma, adafruit:SMA_EDGELAUNCH
- added C17: 0.1uF, MF_Passives:C0402
- added C18, C19: 0.1nF, MF_Passives:C0402
- added R12, R13: 47, MF_Passives:R0402
- added R14: 0, MF_Passives:R0402
- added RFAOUTA+, RFAOUTA-, RFAOUTB+, RFAOUTB-: sma, adafruit:SMA_EDGELAUNCH
- moved J4 4.40 mm to (51.1, 32.4)
- moved R4 4.40 mm to (41.1, 27.4)
- moved R5 4.40 mm to (41.1, 24.4)
- moved R6 4.40 mm to (41.1, 21.4)
- moved R7 4.40 mm to (41.1, 30.4)
- moved C9 4.00 mm to (45.0, 53.0)
- moved C1 2.83 mm to (37.0, 51.0)
Connections:
- new net RFOUTBSMA_N: C18.P$1, RFAOUTB-.P
- new net RFOUTBSMA_P: C19.P$1, RFAOUTB+.P
- new net RFOUTB_N: C18.P$2, R13.P$1, U4.15
- new net RFOUTB_P: C19.P$2, R12.P$1, U4.14
- net +3V3: now also R14.P$1
- net GND: now also C17.P$2, RFAOUTA+.GND@1, RFAOUTA+.GND@2, RFAOUTA+.GND@3, RFAOUTA+.GND@4, RFAOUTA-.GND@1, RFAOUTA-.GND@2, RFAOUTA-.GND@3, RFAOUTA-.GND@4, RFAOUTB+.GND@1, RFAOUTB+.GND@2, RFAOUTB+.GND@3, RFAOUTB+.GND@4, RFAOUTB-.GND@1, RFAOUTB-.GND@2, RFAOUTB-.GND@3, RFAOUTB-.GND@4; no longer RFAOUT+.GND@1, RFAOUT+.GND@2, RFAOUT+.GND@3, RFAOUT+.GND@4, RFAOUT-.GND@1, RFAOUT-.GND@2, RFAOUT-.GND@3, RFAOUT-.GND@4
- net RFOUTASMA_N: now also RFAOUTA-.P; no longer RFAOUT-.P
- net RFOUTASMA_P: now also RFAOUTA+.P; no longer RFAOUT+.P
- net VOUT: now also C17.P$1, R12.P$2, R13.P$2, R14.P$2
Routing:
- net VOUT: track 11.7 -> 35.0 mm, vias 2 -> 4
- net RFOUTB_P: track 0.00 -> 19.8 mm
- net RFOUTB_N: track 0.00 -> 18.1 mm
- net RFOUTBSMA_N: track 0.00 -> 15.8 mm
- net RFOUTBSMA_P: track 0.00 -> 7.25 mm
- net ADFDATA: track 37.6 -> 33.3 mm
- net MUXOUT: track 57.7 -> 53.4 mm
- net ADFCLK: track 40.8 -> 36.5 mm
- net ADFLE: track 34.7 -> 30.3 mm
- net ADFCE: track 30.5 -> 26.1 mm
- net LD: track 62.0 -> 58.1 mm
- net RFOUTASMA_P: track 9.40 -> 6.45 mm
- net +3V3: track 26.2 -> 27.7 mm, vias 7 -> 8
- net GND: track 29.6 -> 30.4 mm, vias 41 -> 60
Other:
- board text added: "Haasoscope Pro Clock board, v1.1 by Dr. Andy Haas September 2024"
- board text removed: "Haasoscope Pro Clock board, v1.0 by Dr. Andy Haas August 2024"
