File: case/back panel.brd (EAGLE design)
At the start: 165 x 30.1 mm, 8 parts, among them J14 2x5, J16 8pin

Commit message: add more connectors
Parts:
- removed J14: 2x5, SparkFun-Connectors:2X5-SHROUDED
Other:
- outline, holes or cut-outs redrawn
- board text added: "Sync IN"
Changed lines of the file:
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@@
 <hole x="2.25" y="3.9" drill="4.5"/>
 <text x="96.628" y="2.011" size="0.8128" layer="21">5V</text>
-<wire x1="84.4" y1="21.75" x2="97.53" y2="21.75" width="0.1524" layer="20"/>
-<wire x1="97.53" y1="21.75" x2="97.53" y2="16" width="0.1524" layer="20"/>
-<wire x1="97.53" y1="16" x2="84.4" y2="16" width="0.1524" layer="20"/>
-<wire x1="84.4" y1="16" x2="84.4" y2="21.75" width="0.1524" layer="20"/>
-<wire x1="69" y1="16" x2="69" y2="19" width="0.1524" layer="21"/>
-<wire x1="91" y1="16" x2="91" y2="19" width="0.1524" layer="21"/>
+<wire x1="73" y1="21.15" x2="83.03" y2="21.15" width="0.1524" layer="20"/>
+<wire x1="83.03" y1="21.15" x2="83.03" y2="16" width="0.1524" layer="20"/>
+<wire x1="83.03" y1="16" x2="73" y2="16" width="0.1524" layer="20"/>
+<wire x1="73" y1="16" x2="73" y2="21.15" width="0.1524" layer="20"/>
 <wire x1="0" y1="16" x2="69" y2="16" width="0.1524" layer="21"/>
-<wire x1="69" y1="16" x2="91" y2="16" width="0.1524" layer="21"/>
-<wire x1="91" y1="16" x2="144.5" y2="16" width="0.1524" layer="21"/>
-<wire x1="144.5" y1="16" x2="160" y2="16" width="0.1524" layer="21"/>
-<wire x1="62.4" y1="21.75" x2="75.53" y2="21.75" width="0.1524" layer="20"/>
-<wire x1="75.53" y1="21.75" x2="75.53" y2="16" width="0.1524" layer="20"/>
-<wire x1="75.53" y1="16" x2="62.4" y2="16" width="0.1524" layer="20"/>
-<wire x1="62.4" y1="16" x2="62.4" y2="21.75" width="0.1524" layer="20"/>
-<text x="37" y="10" size="1.778" layer="21" font="vector">JTAG</text>
+<wire x1="69" y1="16" x2="160" y2="16" width="0.1524" layer="21"/>
+<text x="56.1" y="10.2" size="1.778" layer="21" font="vector">JTAG</text>
 <wire x1="0" y1="7.6" x2="160" y2="7.6" width="0.1524" layer="21"/>
-<text x="87" y="10" size="1.778" layer="21" font="vector">USB C 2.0</text>
-<wire x1="30.1" y1="25.5" x2="50.9" y2="25.5" width="0.1524" layer="20"/>
-<wire x1="50.9" y1="25.5" x2="50.9" y2="15.7" width="0.1524" layer="20"/>
-<wire x1="50.9" y1="15.7" x2="30.2" y2="15.7" width="0.1524" layer="20"/>
-<wire x1="30.2" y1="15.7" x2="30.1" y2="15.8" width="0.1524" layer="20"/>
-<wire x1="30.1" y1="15.8" x2="30.1" y2="25.5" width="0.1524" layer="20"/>
+<text x="73" y="10" size="1.778" layer="21" font="vector">USB C 2.0</text>
+<wire x1="48.6" y1="25.7" x2="69.4" y2="25.7" width="0.1524" layer="20"/>
+<wire x1="69.4" y1="25.7" x2="69.4" y2="15.9" width="0.1524" layer="20"/>
+<wire x1="69.4" y1="15.9" x2="48.7" y2="15.9" width="0.1524" layer="20"/>
+<wire x1="48.7" y1="15.9" x2="48.6" y2="16" width="0.1524" layer="20"/>
+<wire x1="48.6" y1="16" x2="48.6" y2="25.7" width="0.1524" layer="20"/>
+<wire x1="26.2" y1="29.5" x2="41.7" y2="29.5" width="0.1524" layer="20"/>
+<wire x1="41.7" y1="29.5" x2="41.7" y2="16" width="0.1524" layer="20"/>
+<wire x1="41.7" y1="16" x2="26.2" y2="16" width="0.1524" layer="20"/>
+<wire x1="26.2" y1="16" x2="26.1" y2="16.1" width="0.1524" layer="20"/>
+<wire x1="26.1" y1="16.1" x2="26.1" y2="29.4" width="0.1524" layer="20"/>
+<wire x1="26.1" y1="29.4" x2="26.2" y2="29.5" width="0.1524" layer="20"/>
+<text x="28" y="10" size="1.778" layer="21" font="vector">Sync IN</text>
 </plain>
 <attributes>
@@
 <element name="R3" library="FlashPCB_Resistors" package="RES-0402" value="3.3k" x="69.3" y="2.3" smashed="yes"/>
 <element name="R4" library="FlashPCB_Resistors" package="RES-0402" value="3.3k" x="69.3" y="4" smashed="yes"/>
-<element name="J14" library="SparkFun-Connectors" library_urn="urn:adsk.eagle:library:513" package="2X5-SHROUDED" package3d_urn="urn:adsk.eagle:package:38000/1" value="2x5" x="40.5" y="20.6" smashed="yes" rot="R270">
-<attribute name="PROD_ID" value="CONN-08671" x="63.5" y="30.2" size="1.778" layer="27" rot="R270" display="off"/>
-<attribute name="SF_ID" value="PRT-08506" x="63.5" y="30.2" size="1.778" layer="27" rot="R270" display="off"/>
-</element>
 </elements>
 <signals>
@@
 <contactref element="LED2" pad="4"/>
 <contactref element="LED2" pad="6"/>
-<wire x1="96.1" y1="3.6" x2="89.66" y2="4.3" width="0" layer="19" extent="1-1"/>
-<wire x1="62.5" y1="2.3" x2="96.1" y2="3.6" width="0" layer="19" extent="1-1"/>
-<wire x1="62.5" y1="4" x2="62.5" y2="2.3" width="0" layer="19" extent="1-1"/>
+<wire x1="89.66" y1="4.3" x2="96.1" y2="3.6" width="0" layer="19" extent="1-1"/>
+<wire x1="62.5" y1="4" x2="89.66" y2="4.3" width="0" layer="19" extent="1-1"/>
 <wire x1="62.5" y1="5.7" x2="62.5" y2="4" width="0" layer="19" extent="1-1"/>
+<wire x1="62.5" y1="2.3" x2="62.5" y2="4" width="0" layer="19" extent="1-1"/>
 </signal>
 <signal name="SW4">
