File: case/back panel.sch (EAGLE design)
At the start: 8 parts, among them J14 2x5, J16 8pin

Commit message: add more connectors
Parts:
- removed J14: 2x5, SparkFun-Connectors:CONN_05X2SHD
Changed lines of the file:
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@@
 <part name="R3" library="FlashPCB_Resistors" deviceset="RES-0402" device="" value="3.3k"/>
 <part name="R4" library="FlashPCB_Resistors" deviceset="RES-0402" device="" value="3.3k"/>
-<part name="J14" library="SparkFun-Connectors" library_urn="urn:adsk.eagle:library:513" deviceset="CONN_05X2" device="SHD" package3d_urn="urn:adsk.eagle:package:38000/1" value="2x5"/>
 </parts>
 <sheets>
@@
 <attribute name="VALUE" x="49.53" y="23.622" size="1.778" layer="96" rot="R180"/>
 </instance>
-<instance part="J14" gate="G$1" x="129.54" y="22.86" smashed="yes">
-<attribute name="VALUE" x="125.73" y="12.954" size="1.778" layer="96" font="vector"/>
-<attribute name="NAME" x="125.73" y="30.988" size="1.778" layer="95" font="vector"/>
-</instance>
 </instances>

Commit message: move everything down by 3.5mm (one board slot) to make room for eth connectors
Parts:
- removed J16: 8pin, SparkFun-Connectors:CONN_08"
- removed LED1: red, adafruit:LEDCHIP-LED0603
- removed LED2: RGBLED5050, adafruit:RGBLED5050
- removed R1, R2, R3, R4: 3.3k, FlashPCB_Resistors:RES-0402
Connections:
- removed net 5V: J16.1, J16.3, J16.5, J16.7, LED1.A
- removed net BLUE: J16.8, R2.P$2
- removed net BLUE_R: LED2.BLUE_A, R2.P$1
- removed net GND: J16.2, LED2.BLUE_C, LED2.GREEN_C, LED2.RED_C, R1.P$1
- removed net GREEN: J16.6, R3.P$2
- removed net GREEN_R: LED2.GREEN_A, R3.P$1
- removed net N$1: LED1.C, R1.P$2
- removed net RED: J16.4, R4.P$2
- removed net RED_R: LED2.RED_A, R4.P$1
Changed lines of the file:
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@@
 </classes>
 <parts>
-<part name="J16" library="SparkFun-Connectors" library_urn="urn:adsk.eagle:library:513" deviceset="CONN_08" device="&quot;" package3d_urn="urn:adsk.eagle:package:38138/1" value="8pin"/>
-<part name="GND2" library="SparkFun-PowerSymbols" library_urn="urn:adsk.eagle:library:530" deviceset="GND" device=""/>
-<part name="R1" library="FlashPCB_Resistors" deviceset="RES-0402" device="" value="3.3k"/>
-<part name="LED1" library="adafruit" library_urn="urn:adsk.eagle:library:420" deviceset="LED" device="CHIP-LED0603" package3d_urn="urn:adsk.eagle:package:6240556/1" value="red"/>
-<part name="LED2" library="adafruit" library_urn="urn:adsk.eagle:library:420" deviceset="RGBLED" device="5050" package3d_urn="urn:adsk.eagle:package:6240865/1"/>
-<part name="GND1" library="SparkFun-PowerSymbols" library_urn="urn:adsk.eagle:library:530" deviceset="GND" device=""/>
-<part name="R2" library="FlashPCB_Resistors" deviceset="RES-0402" device="" value="3.3k"/>
-<part name="R3" library="FlashPCB_Resistors" deviceset="RES-0402" device="" value="3.3k"/>
-<part name="R4" library="FlashPCB_Resistors" deviceset="RES-0402" device="" value="3.3k"/>
 </parts>
 <sheets>
@@
 </plain>
 <instances>
-<instance part="J16" gate="G$1" x="10.16" y="22.86" smashed="yes" rot="R180"/>
-<instance part="GND2" gate="1" x="93.98" y="7.62" smashed="yes">
-<attribute name="VALUE" x="93.98" y="7.366" size="1.778" layer="96" align="top-center"/>
-</instance>
-<instance part="R1" gate="G$1" x="93.98" y="17.78" smashed="yes" rot="R90">
-<attribute name="NAME" x="92.4814" y="13.97" size="1.778" layer="95" rot="R90"/>
-<attribute name="VALUE" x="97.282" y="13.97" size="1.778" layer="96" rot="R90"/>
-</instance>
-<instance part="LED1" gate="G$1" x="93.98" y="27.94" smashed="yes">
-<attribute name="NAME" x="97.536" y="23.368" size="1.778" layer="95" rot="R90"/>
-<attribute name="VALUE" x="99.695" y="23.368" size="1.778" layer="96" rot="R90"/>
-</instance>
-<instance part="LED2" gate="G$1" x="60.96" y="25.4" smashed="yes">
-<attribute name="NAME" x="57.15" y="34.29" size="1.778" layer="95"/>
-</instance>
-<instance part="GND1" gate="1" x="71.12" y="17.78" smashed="yes">
-<attribute name="VALUE" x="71.12" y="17.526" size="1.778" layer="96" align="top-center"/>
-</instance>
-<instance part="R2" gate="G$1" x="45.72" y="30.48" smashed="yes" rot="R180">
-<attribute name="VALUE" x="49.53" y="33.782" size="1.778" layer="96" rot="R180"/>
-</instance>
-<instance part="R3" gate="G$1" x="45.72" y="25.4" smashed="yes" rot="R180">
-<attribute name="VALUE" x="49.53" y="28.702" size="1.778" layer="96" rot="R180"/>
-</instance>
-<instance part="R4" gate="G$1" x="45.72" y="20.32" smashed="yes" rot="R180">
-<attribute name="VALUE" x="49.53" y="23.622" size="1.778" layer="96" rot="R180"/>
-</instance>
 </instances>
 <busses>
 </busses>
 <nets>
-<net name="GND" class="0">
-<segment>
-<pinref part="GND2" gate="1" pin="GND"/>
-<pinref part="R1" gate="G$1" pin="P$1"/>
-<wire x1="93.98" y1="12.7" x2="93.98" y2="10.16" width="0.1524" layer="91"/>
-</segment>
-<segment>
-<pinref part="J16" gate="G$1" pin="2"/>
-<wire x1="5.08" y1="27.94" x2="-2.54" y2="27.94" width="0.1524" layer="91"/>
-<label x="-2.54" y="27.94" size="1.778" layer="95"/>
-</segment>
-<segment>
-<pinref part="LED2" gate="G$1" pin="RED_C"/>
-<wire x1="66.04" y1="20.32" x2="71.12" y2="20.32" width="0.1524" layer="91"/>
-<pinref part="GND1" gate="1" pin="GND"/>
-<pinref part="LED2" gate="G$1" pin="BLUE_C"/>
-<wire x1="66.04" y1="30.48" x2="71.12" y2="30.48" width="0.1524" layer="91"/>
-<pinref part="LED2" gate="G$1" pin="GREEN_C"/>
-<wire x1="66.04" y1="25.4" x2="71.12" y2="25.4" width="0.1524" layer="91"/>
-<wire x1="71.12" y1="30.48" x2="71.12" y2="25.4" width="0.1524" layer="91"/>
-<wire x1="71.12" y1="25.4" x2="71.12" y2="20.32" width="0.1524" layer="91"/>
-<junction x="71.12" y="25.4"/>
-<junction x="71.12" y="20.32"/>
-</segment>
-</net>
-<net name="5V" class="0">
-<segment>
-<label x="86.36" y="30.48" size="1.778" layer="95"/>
-<wire x1="93.98" y1="30.48" x2="86.36" y2="30.48" width="0.1524" layer="91"/>
-<pinref part="LED1" gate="G$1" pin="A"/>
-</segment>
-<segment>
-<pinref part="J16" gate="G$1" pin="1"/>
-<wire x1="5.08" y1="30.48" x2="-2.54" y2="30.48" width="0.1524" layer="91"/>
-<label x="-2.54" y="30.48" size="1.778" layer="95"/>
-</segment>
-<segment>
-<pinref part="J16" gate="G$1" pin="3"/>
-<wire x1="5.08" y1="25.4" x2="-2.54" y2="25.4" width="0.1524" layer="91"/>
-<label x="-2.54" y="25.4" size="1.778" layer="95"/>
-</segment>
-<segment>
-<pinref part="J16" gate="G$1" pin="5"/>
-<wire x1="5.08" y1="20.32" x2="-2.54" y2="20.32" width="0.1524" layer="91"/>
-<label x="-2.54" y="20.32" size="1.778" layer="95"/>
-</segment>
-<segment>
-<pinref part="J16" gate="G$1" pin="7"/>
-<wire x1="5.08" y1="15.24" x2="-2.54" y2="15.24" width="0.1524" layer="91"/>
-<label x="-2.54" y="15.24" size="1.778" layer="95"/>
-</segment>
-</net>
-<net name="N$1" class="0">
-<segment>
-<pinref part="R1" gate="G$1" pin="P$2"/>
-<pinref part="LED1" gate="G$1" pin="C"/>
-</segment>
-</net>
-<net name="BLUE" class="0">
-<segment>
-<pinref part="J16" gate="G$1" pin="8"/>
-<wire x1="5.08" y1="12.7" x2="-2.54" y2="12.7" width="0.1524" layer="91"/>
-<label x="-2.54" y="12.7" size="1.778" layer="95"/>
-</segment>
-<segment>
-<pinref part="R2" gate="G$1" pin="P$2"/>
-<wire x1="40.64" y1="30.48" x2="30.48" y2="30.48" width="0.1524" layer="91"/>
-<label x="30.48" y="30.48" size="1.778" layer="95"/>
-</segment>
-</net>
-<net name="GREEN" class="0">
-<segment>
-<pinref part="J16" gate="G$1" pin="6"/>
-<wire x1="5.08" y1="17.78" x2="-2.54" y2="17.78" width="0.1524" layer="91"/>
-<label x="-2.54" y="17.78" size="1.778" layer="95"/>
-</segment>
-<segment>
-<pinref part="R3" gate="G$1" pin="P$2"/>
-<wire x1="30.48" y1="25.4" x2="40.64" y2="25.4" width="0.1524" layer="91"/>
-<label x="30.48" y="25.4" size="1.778" layer="95"/>
-</segment>
-</net>
-<net name="RED" class="0">
-<segment>
-<pinref part="J16" gate="G$1" pin="4"/>
-<wire x1="5.08" y1="22.86" x2="-2.54" y2="22.86" width="0.1524" layer="91"/>
-<label x="-2.54" y="22.86" size="1.778" layer="95"/>
-</segment>
-<segment>
-<pinref part="R4" gate="G$1" pin="P$2"/>
-<wire x1="40.64" y1="20.32" x2="30.48" y2="20.32" width="0.1524" layer="91"/>
-<label x="30.48" y="20.32" size="1.778" layer="95"/>
-</segment>
-</net>
-<net name="BLUE_R" class="0">
-<segment>
-<pinref part="LED2" gate="G$1" pin="BLUE_A"/>
-<wire x1="55.88" y1="30.48" x2="50.8" y2="30.48" width="0.1524" layer="91"/>
-<label x="50.8" y="30.48" size="1.778" layer="95"/>
-<pinref part="R2" gate="G$1" pin="P$1"/>
-</segment>
-</net>
-<net name="GREEN_R" class="0">
-<segment>
-<pinref part="LED2" gate="G$1" pin="GREEN_A"/>
-<wire x1="55.88" y1="25.4" x2="50.8" y2="25.4" width="0.1524" layer="91"/>
-<label x="50.8" y="25.4" size="1.778" layer="95"/>
-<pinref part="R3" gate="G$1" pin="P$1"/>
-</segment>
-</net>
-<net name="RED_R" class="0">
-<segment>
-<pinref part="LED2" gate="G$1" pin="RED_A"/>
-<wire x1="55.88" y1="20.32" x2="50.8" y2="20.32" width="0.1524" layer="91"/>
-<label x="50.8" y="20.32" size="1.778" layer="95"/>
-<pinref part="R4" gate="G$1" pin="P$1"/>
-</segment>
-</net>
 </nets>
 </sheet>
@@
 </schematic>
 </drawing>
-<compatibility>
-<note version="8.2" severity="warning">
-Since Version 8.2, EAGLE supports online libraries. The ids
-of those online libraries will not be understood (or retained)
-with this version.
-</note>
-<note version="8.3" severity="warning">
-Since Version 8.3, EAGLE supports URNs for individual library
-assets (packages, symbols, and devices). The URNs of those assets
-will not be understood (or retained) with this version.
-</note>
-<note version="8.3" severity="warning">
-Since Version 8.3, EAGLE supports the association of 3D packages
-with devices in libraries, schematics, and board files. Those 3D
-packages will not be understood (or retained) with this version.
-</note>
-</compatibility>
 </eagle>

Commit message: v1.00
Parts:
- added C2: 10uF, Nordic_nRF:CAPACITOR_0805_N
- added D1: green, MF_LEDs:LED_SINGLE-0805
- added R1: 3.3k, FlashPCB_Resistors:RES-0402
Connections:
- new net 5V: C2.1, D1.ANODE
- new net GND: C2.2, R1.P$1
- new net N$7: D1.CATHODE, R1.P$2
Changed lines of the file:
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@@
 </classes>
 <parts>
+<part name="D1" library="MF_LEDs" deviceset="LED_SINGLE" device="-0805" value="green"/>
+<part name="R1" library="FlashPCB_Resistors" deviceset="RES-0402" device="" value="3.3k"/>
+<part name="C2" library="Nordic_nRF" library_urn="urn:adsk.eagle:library:169009" deviceset="CAPACITOR" device="_0805_N" package3d_urn="urn:adsk.eagle:package:2593736/1" value="10uF"/>
 </parts>
 <sheets>
@@
 </plain>
 <instances>
+<instance part="D1" gate="G$1" x="66.04" y="66.04" smashed="yes" rot="R270">
+<attribute name="NAME" x="63.5" y="68.58" size="1.016" layer="95" font="vector" rot="R270" align="top-left"/>
+<attribute name="VALUE" x="60.96" y="68.58" size="1.016" layer="96" font="vector" rot="R270"/>
+</instance>
+<instance part="R1" gate="G$1" x="66.04" y="58.42" smashed="yes" rot="R90">
+<attribute name="NAME" x="64.5414" y="54.61" size="1.778" layer="95" rot="R90"/>
+<attribute name="VALUE" x="69.342" y="54.61" size="1.778" layer="96" rot="R90"/>
+</instance>
+<instance part="C2" gate="C$1" x="50.8" y="66.04" smashed="yes">
+<attribute name="NAME" x="52.324" y="68.961" size="1.778" layer="95"/>
+<attribute name="VALUE" x="52.324" y="64.389" size="1.778" layer="96"/>
+</instance>
 </instances>
 <busses>
 </busses>
 <nets>
+<net name="GND" class="0">
+<segment>
+<pinref part="R1" gate="G$1" pin="P$1"/>
+<wire x1="66.04" y1="53.34" x2="50.8" y2="53.34" width="0.1524" layer="91"/>
+<wire x1="50.8" y1="53.34" x2="40.64" y2="53.34" width="0.1524" layer="91"/>
+<wire x1="50.8" y1="60.96" x2="50.8" y2="53.34" width="0.1524" layer="91"/>
+<junction x="50.8" y="53.34"/>
+<pinref part="C2" gate="C$1" pin="2"/>
+<label x="40.64" y="53.34" size="1.778" layer="95"/>
+</segment>
+</net>
+<net name="5V" class="0">
+<segment>
+<pinref part="D1" gate="G$1" pin="ANODE"/>
+<wire x1="66.04" y1="68.58" x2="50.8" y2="68.58" width="0.1524" layer="91"/>
+<pinref part="C2" gate="C$1" pin="1"/>
+<wire x1="50.8" y1="68.58" x2="40.64" y2="68.58" width="0.1524" layer="91"/>
+<junction x="50.8" y="68.58"/>
+<label x="40.64" y="68.58" size="1.778" layer="95"/>
+</segment>
+</net>
+<net name="N$7" class="0">
+<segment>
+<pinref part="D1" gate="G$1" pin="CATHODE"/>
+<pinref part="R1" gate="G$1" pin="P$2"/>
+</segment>
+</net>
 </nets>
 </sheet>
 </sheets>
+<errors>
+</errors>
 </schematic>
 </drawing>
+<compatibility>
+<note version="8.2" severity="warning">
+Since Version 8.2, EAGLE supports online libraries. The ids
+of those online libraries will not be understood (or retained)
+with this version.
+</note>
+<note version="8.3" severity="warning">
+Since Version 8.3, EAGLE supports URNs for individual library
+assets (packages, symbols, and devices). The URNs of those assets
+will not be understood (or retained) with this version.
+</note>
+<note version="8.3" severity="warning">
+Since Version 8.3, EAGLE supports the association of 3D packages
+with devices in libraries, schematics, and board files. Those 3D
+packages will not be understood (or retained) with this version.
+</note>
+</compatibility>
 </eagle>
