File: case/front panel.sch (EAGLE design)
At the start: 3 parts, among them J16 8pin

Commit message: front panel pcb v1.0
Parts:
- added LED2: RGBLED5050, adafruit:RGBLED5050
- added R2, R3, R4: 3.3k, FlashPCB_Resistors:RES-0402
Connections:
- new net BLUE: J16.8, R2.P$2
- new net BLUE_R: LED2.BLUE_A, R2.P$1
- new net GREEN: J16.6, R3.P$2
- new net GREEN_R: LED2.GREEN_A, R3.P$1
- new net RED: J16.4, R4.P$2
- new net RED_R: LED2.RED_A, R4.P$1
- net 5V: now also J16.3, J16.5, J16.7
- net GND: now also LED2.BLUE_C, LED2.GREEN_C, LED2.RED_C
Changed lines of the file:
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@@
 <part name="R1" library="FlashPCB_Resistors" deviceset="RES-0402" device="" value="3.3k"/>
 <part name="LED1" library="adafruit" library_urn="urn:adsk.eagle:library:420" deviceset="LED" device="CHIP-LED0603" package3d_urn="urn:adsk.eagle:package:6240556/1" value="red"/>
+<part name="LED2" library="adafruit" library_urn="urn:adsk.eagle:library:420" deviceset="RGBLED" device="5050" package3d_urn="urn:adsk.eagle:package:6240865/1"/>
+<part name="GND1" library="SparkFun-PowerSymbols" library_urn="urn:adsk.eagle:library:530" deviceset="GND" device=""/>
+<part name="R2" library="FlashPCB_Resistors" deviceset="RES-0402" device="" value="3.3k"/>
+<part name="R3" library="FlashPCB_Resistors" deviceset="RES-0402" device="" value="3.3k"/>
+<part name="R4" library="FlashPCB_Resistors" deviceset="RES-0402" device="" value="3.3k"/>
 </parts>
 <sheets>
@@
 </plain>
 <instances>
-<instance part="J16" gate="G$1" x="35.56" y="20.32" smashed="yes" rot="R180"/>
+<instance part="J16" gate="G$1" x="10.16" y="22.86" smashed="yes" rot="R180"/>
 <instance part="GND2" gate="1" x="93.98" y="7.62" smashed="yes">
 <attribute name="VALUE" x="93.98" y="7.366" size="1.778" layer="96" align="top-center"/>
@@
 <attribute name="NAME" x="97.536" y="23.368" size="1.778" layer="95" rot="R90"/>
 <attribute name="VALUE" x="99.695" y="23.368" size="1.778" layer="96" rot="R90"/>
+</instance>
+<instance part="LED2" gate="G$1" x="60.96" y="25.4" smashed="yes">
+<attribute name="NAME" x="57.15" y="34.29" size="1.778" layer="95"/>
+</instance>
+<instance part="GND1" gate="1" x="71.12" y="17.78" smashed="yes">
+<attribute name="VALUE" x="71.12" y="17.526" size="1.778" layer="96" align="top-center"/>
+</instance>
+<instance part="R2" gate="G$1" x="45.72" y="30.48" smashed="yes" rot="R180">
+<attribute name="VALUE" x="49.53" y="33.782" size="1.778" layer="96" rot="R180"/>
+</instance>
+<instance part="R3" gate="G$1" x="45.72" y="25.4" smashed="yes" rot="R180">
+<attribute name="VALUE" x="49.53" y="28.702" size="1.778" layer="96" rot="R180"/>
+</instance>
+<instance part="R4" gate="G$1" x="45.72" y="20.32" smashed="yes" rot="R180">
+<attribute name="VALUE" x="49.53" y="23.622" size="1.778" layer="96" rot="R180"/>
 </instance>
 </instances>
@@
 <segment>
 <pinref part="J16" gate="G$1" pin="2"/>
-<wire x1="30.48" y1="25.4" x2="22.86" y2="25.4" width="0.1524" layer="91"/>
-<label x="22.86" y="25.4" size="1.778" layer="95"/>
+<wire x1="5.08" y1="27.94" x2="-2.54" y2="27.94" width="0.1524" layer="91"/>
+<label x="-2.54" y="27.94" size="1.778" layer="95"/>
+</segment>
+<segment>
+<pinref part="LED2" gate="G$1" pin="RED_C"/>
+<wire x1="66.04" y1="20.32" x2="71.12" y2="20.32" width="0.1524" layer="91"/>
+<pinref part="GND1" gate="1" pin="GND"/>
+<pinref part="LED2" gate="G$1" pin="BLUE_C"/>
+<wire x1="66.04" y1="30.48" x2="71.12" y2="30.48" width="0.1524" layer="91"/>
+<pinref part="LED2" gate="G$1" pin="GREEN_C"/>
+<wire x1="66.04" y1="25.4" x2="71.12" y2="25.4" width="0.1524" layer="91"/>
+<wire x1="71.12" y1="30.48" x2="71.12" y2="25.4" width="0.1524" layer="91"/>
+<wire x1="71.12" y1="25.4" x2="71.12" y2="20.32" width="0.1524" layer="91"/>
+<junction x="71.12" y="25.4"/>
+<junction x="71.12" y="20.32"/>
 </segment>
 </net>
@@
 <segment>
 <pinref part="J16" gate="G$1" pin="1"/>
-<wire x1="30.48" y1="27.94" x2="22.86" y2="27.94" width="0.1524" layer="91"/>
-<label x="22.86" y="27.94" size="1.778" layer="95"/>
+<wire x1="5.08" y1="30.48" x2="-2.54" y2="30.48" width="0.1524" layer="91"/>
+<label x="-2.54" y="30.48" size="1.778" layer="95"/>
+</segment>
+<segment>
+<pinref part="J16" gate="G$1" pin="3"/>
+<wire x1="5.08" y1="25.4" x2="-2.54" y2="25.4" width="0.1524" layer="91"/>
+<label x="-2.54" y="25.4" size="1.778" layer="95"/>
+</segment>
+<segment>
+<pinref part="J16" gate="G$1" pin="5"/>
+<wire x1="5.08" y1="20.32" x2="-2.54" y2="20.32" width="0.1524" layer="91"/>
+<label x="-2.54" y="20.32" size="1.778" layer="95"/>
+</segment>
+<segment>
+<pinref part="J16" gate="G$1" pin="7"/>
+<wire x1="5.08" y1="15.24" x2="-2.54" y2="15.24" width="0.1524" layer="91"/>
+<label x="-2.54" y="15.24" size="1.778" layer="95"/>
 </segment>
 </net>
@@
 </segment>
 </net>
+<net name="BLUE" class="0">
+<segment>
+<pinref part="J16" gate="G$1" pin="8"/>
+<wire x1="5.08" y1="12.7" x2="-2.54" y2="12.7" width="0.1524" layer="91"/>
+<label x="-2.54" y="12.7" size="1.778" layer="95"/>
+</segment>
+<segment>
+<pinref part="R2" gate="G$1" pin="P$2"/>
+<wire x1="40.64" y1="30.48" x2="30.48" y2="30.48" width="0.1524" layer="91"/>
+<label x="30.48" y="30.48" size="1.778" layer="95"/>
+</segment>
+</net>
+<net name="GREEN" class="0">
+<segment>
+<pinref part="J16" gate="G$1" pin="6"/>
+<wire x1="5.08" y1="17.78" x2="-2.54" y2="17.78" width="0.1524" layer="91"/>
+<label x="-2.54" y="17.78" size="1.778" layer="95"/>
+</segment>
+<segment>
+<pinref part="R3" gate="G$1" pin="P$2"/>
+<wire x1="30.48" y1="25.4" x2="40.64" y2="25.4" width="0.1524" layer="91"/>
+<label x="30.48" y="25.4" size="1.778" layer="95"/>
+</segment>
+</net>
+<net name="RED" class="0">
+<segment>
+<pinref part="J16" gate="G$1" pin="4"/>
+<wire x1="5.08" y1="22.86" x2="-2.54" y2="22.86" width="0.1524" layer="91"/>
+<label x="-2.54" y="22.86" size="1.778" layer="95"/>
+</segment>
+<segment>
+<pinref part="R4" gate="G$1" pin="P$2"/>
+<wire x1="40.64" y1="20.32" x2="30.48" y2="20.32" width="0.1524" layer="91"/>
+<label x="30.48" y="20.32" size="1.778" layer="95"/>
+</segment>
+</net>
+<net name="BLUE_R" class="0">
+<segment>
+<pinref part="LED2" gate="G$1" pin="BLUE_A"/>
+<wire x1="55.88" y1="30.48" x2="50.8" y2="30.48" width="0.1524" layer="91"/>
+<label x="50.8" y="30.48" size="1.778" layer="95"/>
+<pinref part="R2" gate="G$1" pin="P$1"/>
+</segment>
+</net>
+<net name="GREEN_R" class="0">
+<segment>
+<pinref part="LED2" gate="G$1" pin="GREEN_A"/>
+<wire x1="55.88" y1="25.4" x2="50.8" y2="25.4" width="0.1524" layer="91"/>
+<label x="50.8" y="25.4" size="1.778" layer="95"/>
+<pinref part="R3" gate="G$1" pin="P$1"/>
+</segment>
+</net>
+<net name="RED_R" class="0">
+<segment>
+<pinref part="LED2" gate="G$1" pin="RED_A"/>
+<wire x1="55.88" y1="20.32" x2="50.8" y2="20.32" width="0.1524" layer="91"/>
+<label x="50.8" y="20.32" size="1.778" layer="95"/>
+<pinref part="R4" gate="G$1" pin="P$1"/>
+</segment>
+</net>

Commit message: move everything down by 3.5mm (one board slot) to make room for eth connectors
Parts:
- removed J16: 8pin, SparkFun-Connectors:CONN_08"
- removed LED1: red, adafruit:LEDCHIP-LED0603
- removed LED2: RGBLED5050, adafruit:RGBLED5050
- removed R1, R2, R3, R4: 3.3k, FlashPCB_Resistors:RES-0402
Connections:
- removed net 5V: J16.1, J16.3, J16.5, J16.7, LED1.A
- removed net BLUE: J16.8, R2.P$2
- removed net BLUE_R: LED2.BLUE_A, R2.P$1
- removed net GND: J16.2, LED2.BLUE_C, LED2.GREEN_C, LED2.RED_C, R1.P$1
- removed net GREEN: J16.6, R3.P$2
- removed net GREEN_R: LED2.GREEN_A, R3.P$1
- removed net N$1: LED1.C, R1.P$2
- removed net RED: J16.4, R4.P$2
- removed net RED_R: LED2.RED_A, R4.P$1
Changed lines of the file:
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@@
 </classes>
 <parts>
-<part name="J16" library="SparkFun-Connectors" library_urn="urn:adsk.eagle:library:513" deviceset="CONN_08" device="&quot;" package3d_urn="urn:adsk.eagle:package:38138/1" value="8pin"/>
-<part name="GND2" library="SparkFun-PowerSymbols" library_urn="urn:adsk.eagle:library:530" deviceset="GND" device=""/>
-<part name="R1" library="FlashPCB_Resistors" deviceset="RES-0402" device="" value="3.3k"/>
-<part name="LED1" library="adafruit" library_urn="urn:adsk.eagle:library:420" deviceset="LED" device="CHIP-LED0603" package3d_urn="urn:adsk.eagle:package:6240556/1" value="red"/>
-<part name="LED2" library="adafruit" library_urn="urn:adsk.eagle:library:420" deviceset="RGBLED" device="5050" package3d_urn="urn:adsk.eagle:package:6240865/1"/>
-<part name="GND1" library="SparkFun-PowerSymbols" library_urn="urn:adsk.eagle:library:530" deviceset="GND" device=""/>
-<part name="R2" library="FlashPCB_Resistors" deviceset="RES-0402" device="" value="3.3k"/>
-<part name="R3" library="FlashPCB_Resistors" deviceset="RES-0402" device="" value="3.3k"/>
-<part name="R4" library="FlashPCB_Resistors" deviceset="RES-0402" device="" value="3.3k"/>
 </parts>
 <sheets>
@@
 </plain>
 <instances>
-<instance part="J16" gate="G$1" x="10.16" y="22.86" smashed="yes" rot="R180"/>
-<instance part="GND2" gate="1" x="93.98" y="7.62" smashed="yes">
-<attribute name="VALUE" x="93.98" y="7.366" size="1.778" layer="96" align="top-center"/>
-</instance>
-<instance part="R1" gate="G$1" x="93.98" y="17.78" smashed="yes" rot="R90">
-<attribute name="NAME" x="92.4814" y="13.97" size="1.778" layer="95" rot="R90"/>
-<attribute name="VALUE" x="97.282" y="13.97" size="1.778" layer="96" rot="R90"/>
-</instance>
-<instance part="LED1" gate="G$1" x="93.98" y="27.94" smashed="yes">
-<attribute name="NAME" x="97.536" y="23.368" size="1.778" layer="95" rot="R90"/>
-<attribute name="VALUE" x="99.695" y="23.368" size="1.778" layer="96" rot="R90"/>
-</instance>
-<instance part="LED2" gate="G$1" x="60.96" y="25.4" smashed="yes">
-<attribute name="NAME" x="57.15" y="34.29" size="1.778" layer="95"/>
-</instance>
-<instance part="GND1" gate="1" x="71.12" y="17.78" smashed="yes">
-<attribute name="VALUE" x="71.12" y="17.526" size="1.778" layer="96" align="top-center"/>
-</instance>
-<instance part="R2" gate="G$1" x="45.72" y="30.48" smashed="yes" rot="R180">
-<attribute name="VALUE" x="49.53" y="33.782" size="1.778" layer="96" rot="R180"/>
-</instance>
-<instance part="R3" gate="G$1" x="45.72" y="25.4" smashed="yes" rot="R180">
-<attribute name="VALUE" x="49.53" y="28.702" size="1.778" layer="96" rot="R180"/>
-</instance>
-<instance part="R4" gate="G$1" x="45.72" y="20.32" smashed="yes" rot="R180">
-<attribute name="VALUE" x="49.53" y="23.622" size="1.778" layer="96" rot="R180"/>
-</instance>
 </instances>
 <busses>
 </busses>
 <nets>
-<net name="GND" class="0">
-<segment>
-<pinref part="GND2" gate="1" pin="GND"/>
-<pinref part="R1" gate="G$1" pin="P$1"/>
-<wire x1="93.98" y1="12.7" x2="93.98" y2="10.16" width="0.1524" layer="91"/>
-</segment>
-<segment>
-<pinref part="J16" gate="G$1" pin="2"/>
-<wire x1="5.08" y1="27.94" x2="-2.54" y2="27.94" width="0.1524" layer="91"/>
-<label x="-2.54" y="27.94" size="1.778" layer="95"/>
-</segment>
-<segment>
-<pinref part="LED2" gate="G$1" pin="RED_C"/>
-<wire x1="66.04" y1="20.32" x2="71.12" y2="20.32" width="0.1524" layer="91"/>
-<pinref part="GND1" gate="1" pin="GND"/>
-<pinref part="LED2" gate="G$1" pin="BLUE_C"/>
-<wire x1="66.04" y1="30.48" x2="71.12" y2="30.48" width="0.1524" layer="91"/>
-<pinref part="LED2" gate="G$1" pin="GREEN_C"/>
-<wire x1="66.04" y1="25.4" x2="71.12" y2="25.4" width="0.1524" layer="91"/>
-<wire x1="71.12" y1="30.48" x2="71.12" y2="25.4" width="0.1524" layer="91"/>
-<wire x1="71.12" y1="25.4" x2="71.12" y2="20.32" width="0.1524" layer="91"/>
-<junction x="71.12" y="25.4"/>
-<junction x="71.12" y="20.32"/>
-</segment>
-</net>
-<net name="5V" class="0">
-<segment>
-<label x="86.36" y="30.48" size="1.778" layer="95"/>
-<wire x1="93.98" y1="30.48" x2="86.36" y2="30.48" width="0.1524" layer="91"/>
-<pinref part="LED1" gate="G$1" pin="A"/>
-</segment>
-<segment>
-<pinref part="J16" gate="G$1" pin="1"/>
-<wire x1="5.08" y1="30.48" x2="-2.54" y2="30.48" width="0.1524" layer="91"/>
-<label x="-2.54" y="30.48" size="1.778" layer="95"/>
-</segment>
-<segment>
-<pinref part="J16" gate="G$1" pin="3"/>
-<wire x1="5.08" y1="25.4" x2="-2.54" y2="25.4" width="0.1524" layer="91"/>
-<label x="-2.54" y="25.4" size="1.778" layer="95"/>
-</segment>
-<segment>
-<pinref part="J16" gate="G$1" pin="5"/>
-<wire x1="5.08" y1="20.32" x2="-2.54" y2="20.32" width="0.1524" layer="91"/>
-<label x="-2.54" y="20.32" size="1.778" layer="95"/>
-</segment>
-<segment>
-<pinref part="J16" gate="G$1" pin="7"/>
-<wire x1="5.08" y1="15.24" x2="-2.54" y2="15.24" width="0.1524" layer="91"/>
-<label x="-2.54" y="15.24" size="1.778" layer="95"/>
-</segment>
-</net>
-<net name="N$1" class="0">
-<segment>
-<pinref part="R1" gate="G$1" pin="P$2"/>
-<pinref part="LED1" gate="G$1" pin="C"/>
-</segment>
-</net>
-<net name="BLUE" class="0">
-<segment>
-<pinref part="J16" gate="G$1" pin="8"/>
-<wire x1="5.08" y1="12.7" x2="-2.54" y2="12.7" width="0.1524" layer="91"/>
-<label x="-2.54" y="12.7" size="1.778" layer="95"/>
-</segment>
-<segment>
-<pinref part="R2" gate="G$1" pin="P$2"/>
-<wire x1="40.64" y1="30.48" x2="30.48" y2="30.48" width="0.1524" layer="91"/>
-<label x="30.48" y="30.48" size="1.778" layer="95"/>
-</segment>
-</net>
-<net name="GREEN" class="0">
-<segment>
-<pinref part="J16" gate="G$1" pin="6"/>
-<wire x1="5.08" y1="17.78" x2="-2.54" y2="17.78" width="0.1524" layer="91"/>
-<label x="-2.54" y="17.78" size="1.778" layer="95"/>
-</segment>
-<segment>
-<pinref part="R3" gate="G$1" pin="P$2"/>
-<wire x1="30.48" y1="25.4" x2="40.64" y2="25.4" width="0.1524" layer="91"/>
-<label x="30.48" y="25.4" size="1.778" layer="95"/>
-</segment>
-</net>
-<net name="RED" class="0">
-<segment>
-<pinref part="J16" gate="G$1" pin="4"/>
-<wire x1="5.08" y1="22.86" x2="-2.54" y2="22.86" width="0.1524" layer="91"/>
-<label x="-2.54" y="22.86" size="1.778" layer="95"/>
-</segment>
-<segment>
-<pinref part="R4" gate="G$1" pin="P$2"/>
-<wire x1="40.64" y1="20.32" x2="30.48" y2="20.32" width="0.1524" layer="91"/>
-<label x="30.48" y="20.32" size="1.778" layer="95"/>
-</segment>
-</net>
-<net name="BLUE_R" class="0">
-<segment>
-<pinref part="LED2" gate="G$1" pin="BLUE_A"/>
-<wire x1="55.88" y1="30.48" x2="50.8" y2="30.48" width="0.1524" layer="91"/>
-<label x="50.8" y="30.48" size="1.778" layer="95"/>
-<pinref part="R2" gate="G$1" pin="P$1"/>
-</segment>
-</net>
-<net name="GREEN_R" class="0">
-<segment>
-<pinref part="LED2" gate="G$1" pin="GREEN_A"/>
-<wire x1="55.88" y1="25.4" x2="50.8" y2="25.4" width="0.1524" layer="91"/>
-<label x="50.8" y="25.4" size="1.778" layer="95"/>
-<pinref part="R3" gate="G$1" pin="P$1"/>
-</segment>
-</net>
-<net name="RED_R" class="0">
-<segment>
-<pinref part="LED2" gate="G$1" pin="RED_A"/>
-<wire x1="55.88" y1="20.32" x2="50.8" y2="20.32" width="0.1524" layer="91"/>
-<label x="50.8" y="20.32" size="1.778" layer="95"/>
-<pinref part="R4" gate="G$1" pin="P$1"/>
-</segment>
-</net>
 </nets>
 </sheet>
@@
 </schematic>
 </drawing>
-<compatibility>
-<note version="8.2" severity="warning">
-Since Version 8.2, EAGLE supports online libraries. The ids
-of those online libraries will not be understood (or retained)
-with this version.
-</note>
-<note version="8.3" severity="warning">
-Since Version 8.3, EAGLE supports URNs for individual library
-assets (packages, symbols, and devices). The URNs of those assets
-will not be understood (or retained) with this version.
-</note>
-<note version="8.3" severity="warning">
-Since Version 8.3, EAGLE supports the association of 3D packages
-with devices in libraries, schematics, and board files. Those 3D
-packages will not be understood (or retained) with this version.
-</note>
-</compatibility>
 </eagle>

Commit message: v1.00
Parts:
- added C1: 10uF, Nordic_nRF:CAPACITOR_0805_N
- added D2: green, MF_LEDs:LED_SINGLE-0805
- added R2: 3.3k, FlashPCB_Resistors:RES-0402
Connections:
- new net 5V: C1.1, D2.ANODE
- new net GND: C1.2, R2.P$1
- new net N$2: D2.CATHODE, R2.P$2
Changed lines of the file:
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@@
 <layer number="56" name="wert" color="7" fill="1" visible="no" active="no"/>
 <layer number="57" name="tCAD" color="7" fill="1" visible="no" active="no"/>
+<layer number="58" name="bCAD" color="11" fill="1" visible="no" active="no"/>
 <layer number="59" name="tCarbon" color="7" fill="1" visible="no" active="no"/>
 <layer number="60" name="bCarbon" color="7" fill="1" visible="no" active="no"/>
@@
 <layer number="136" name="silktop" color="7" fill="1" visible="yes" active="yes"/>
 <layer number="137" name="silkbottom" color="7" fill="1" visible="yes" active="yes"/>
+<layer number="138" name="EEE" color="7" fill="1" visible="no" active="yes"/>
+<layer number="139" name="_tKeepout" color="7" fill="1" visible="no" active="yes"/>
+<layer number="140" name="mbKeepout" color="7" fill="1" visible="no" active="yes"/>
+<layer number="141" name="ASSEMBLY_TOP" color="7" fill="1" visible="no" active="yes"/>
+<layer number="142" name="mbRestrict" color="7" fill="1" visible="no" active="yes"/>
+<layer number="143" name="PLACE_BOUND_TOP" color="7" fill="1" visible="no" active="yes"/>
 <layer number="144" name="Drill_legend" color="7" fill="1" visible="yes" active="yes"/>
 <layer number="145" name="DrillLegend_01-16" color="7" fill="1" visible="yes" active="yes"/>
 <layer number="146" name="DrillLegend_01-20" color="7" fill="1" visible="yes" active="yes"/>
+<layer number="147" name="PIN_NUMBER" color="7" fill="1" visible="no" active="yes"/>
+<layer number="148" name="mDocument" color="7" fill="1" visible="no" active="yes"/>
+<layer number="149" name="DrillLegend_02-15" color="7" fill="1" visible="no" active="yes"/>
 <layer number="150" name="Notes" color="7" fill="1" visible="yes" active="yes"/>
 <layer number="151" name="HeatSink" color="7" fill="1" visible="yes" active="yes"/>
@@
 <layer number="166" name="AntennaArea" color="7" fill="1" visible="yes" active="yes"/>
 <layer number="168" name="4mmHeightArea" color="7" fill="1" visible="yes" active="yes"/>
+<layer number="191" name="mNets" color="7" fill="1" visible="no" active="yes"/>
+<layer number="192" name="mBusses" color="7" fill="1" visible="no" active="yes"/>
+<layer number="193" name="mPins" color="7" fill="1" visible="no" active="yes"/>
+<layer number="194" name="mSymbols" color="7" fill="1" visible="no" active="yes"/>
+<layer number="195" name="mNames" color="7" fill="1" visible="no" active="yes"/>
+<layer number="196" name="mValues" color="7" fill="1" visible="no" active="yes"/>
 <layer number="199" name="Contour" color="7" fill="1" visible="yes" active="yes"/>
 <layer number="200" name="200bmp" color="1" fill="10" visible="yes" active="yes"/>
@@
 </classes>
 <parts>
+<part name="D2" library="MF_LEDs" deviceset="LED_SINGLE" device="-0805" value="green"/>
+<part name="R2" library="FlashPCB_Resistors" deviceset="RES-0402" device="" value="3.3k"/>
+<part name="C1" library="Nordic_nRF" library_urn="urn:adsk.eagle:library:169009" deviceset="CAPACITOR" device="_0805_N" package3d_urn="urn:adsk.eagle:package:2593736/1" value="10uF"/>
 </parts>
 <sheets>
@@
 </plain>
 <instances>
+<instance part="D2" gate="G$1" x="38.1" y="27.94" smashed="yes" rot="R270">
+<attribute name="NAME" x="35.56" y="30.48" size="1.016" layer="95" font="vector" rot="R270" align="top-left"/>
+<attribute name="VALUE" x="33.02" y="30.48" size="1.016" layer="96" font="vector" rot="R270"/>
+</instance>
+<instance part="R2" gate="G$1" x="38.1" y="20.32" smashed="yes" rot="R90">
+<attribute name="NAME" x="36.6014" y="16.51" size="1.778" layer="95" rot="R90"/>
+<attribute name="VALUE" x="41.402" y="16.51" size="1.778" layer="96" rot="R90"/>
+</instance>
+<instance part="C1" gate="C$1" x="22.86" y="27.94" smashed="yes">
+<attribute name="NAME" x="24.384" y="30.861" size="1.778" layer="95"/>
+<attribute name="VALUE" x="24.384" y="26.289" size="1.778" layer="96"/>
+</instance>
 </instances>
 <busses>
 </busses>
 <nets>
+<net name="GND" class="0">
+<segment>
+<pinref part="R2" gate="G$1" pin="P$1"/>
+<wire x1="38.1" y1="15.24" x2="22.86" y2="15.24" width="0.1524" layer="91"/>
+<wire x1="22.86" y1="15.24" x2="12.7" y2="15.24" width="0.1524" layer="91"/>
+<wire x1="22.86" y1="22.86" x2="22.86" y2="15.24" width="0.1524" layer="91"/>
+<junction x="22.86" y="15.24"/>
+<pinref part="C1" gate="C$1" pin="2"/>
+<label x="12.7" y="15.24" size="1.778" layer="95"/>
+</segment>
+</net>
+<net name="5V" class="0">
+<segment>
+<pinref part="D2" gate="G$1" pin="ANODE"/>
+<wire x1="38.1" y1="30.48" x2="22.86" y2="30.48" width="0.1524" layer="91"/>
+<pinref part="C1" gate="C$1" pin="1"/>
+<wire x1="22.86" y1="30.48" x2="12.7" y2="30.48" width="0.1524" layer="91"/>
+<junction x="22.86" y="30.48"/>
+<label x="12.7" y="30.48" size="1.778" layer="95"/>
+</segment>
+</net>
+<net name="N$1" class="0">
+</net>
+<net name="N$2" class="0">
+<segment>
+<pinref part="R2" gate="G$1" pin="P$2"/>
+<pinref part="D2" gate="G$1" pin="CATHODE"/>
+</segment>
+</net>
 </nets>
 </sheet>
 </sheets>
+<errors>
+</errors>
 </schematic>
 </drawing>
+<compatibility>
+<note version="8.2" severity="warning">
+Since Version 8.2, EAGLE supports online libraries. The ids
+of those online libraries will not be understood (or retained)
+with this version.
+</note>
+<note version="8.3" severity="warning">
+Since Version 8.3, EAGLE supports URNs for individual library
+assets (packages, symbols, and devices). The URNs of those assets
+will not be understood (or retained) with this version.
+</note>
+<note version="8.3" severity="warning">
+Since Version 8.3, EAGLE supports the association of 3D packages
+with devices in libraries, schematics, and board files. Those 3D
+packages will not be understood (or retained) with this version.
+</note>
+</compatibility>
 </eagle>
